Commit message: Unify autonomous exploration into launch_sim and tune robot configs

File: description/lidar.xacro (robot description, xacro)
@@ -66,5 +66,5 @@
     <!-- Ignition Gazebo Sensors Plugin (required to activate sensors) -->
     <gazebo>
-        <plugin filename="libignition-gazebo-sensors-system.so" name="ignition::gazebo::systems::Sensors">
+        <plugin filename="libgz-sim-sensors-system.so" name="gz::sim::systems::Sensors">
             <render_engine>ogre2</render_engine>
         </plugin>

File: description/robot_core.xacro (robot description, xacro)
@@ -105,9 +105,9 @@
     <parent link = "chassis"/>
     <child link = "caster_wheel"/>
-    <origin xyz = "0.1 0 0" rpy = "0 0 0"/>
+    <origin xyz = "-0.15 0 0.025" rpy = "0 0 0"/>
 </joint>
 <link name = "caster_wheel">
     <visual>
-        <origin xyz = "0.3 0 0"/>
+        <origin xyz = "0 0 0"/>
         <geometry>
             <sphere radius = "0.05"/>
@@ -118,5 +118,5 @@
     </visual>
     <collision>
-        <origin xyz = "0.3 0 0"/>
+        <origin xyz = "0 0 0"/>
         <geometry>
             <sphere radius = "0.05"/>
@@ -124,5 +124,5 @@
     </collision>
     <xacro:inertial_sphere mass = "0.04" radius="0.05">
-        <origin xyz ="0.3 0 0" rpy="0 0 0"/>
+        <origin xyz ="0 0 0" rpy="0 0 0"/>
     </xacro:inertial_sphere>
 </link>

Commit message: updated

File: description/lidar.xacro (robot description, xacro)
@@ -2,5 +2,5 @@
 <robot xmlns:xacro="http://www.ros.org/wiki/xacro">
     <!-- LIDAR SENSOR -->
-    <!-- Lidar Joint -->
+    <!-- Lidar Joint — fixed mount on top of chassis -->
     <joint name="laser_joint" type="fixed">
         <parent link="chassis"/>
@@ -29,9 +29,11 @@
         </inertial>
     </link>
-    <!-- Gazebo Lidar Color -->
-    <gazebo reference="laser_frame">
-        <material>Gazebo/Black</material>
-    </gazebo>
-    <!-- Ignition Gazebo Lidar Plugin (GPU Lidar sensor) -->
+    <!--
+        Ignition Gazebo GPU LiDAR sensor.
+        • topic="scan"  → bridged to ROS as /scan
+        • <ignition_frame_id> sets the frame_id in the ROS LaserScan header.
+          USE <ignition_frame_id> for Ignition Gazebo 6 (Fortress) + ROS2 Humble.
+          <gz_frame_id> is for the newer Gazebo (Harmonic+) and will be IGNORED here.
+    -->
     <gazebo reference="laser_frame">
         <sensor name="gpu_lidar" type="gpu_lidar">
@@ -64,7 +66,12 @@
         </sensor>
     </gazebo>
-    <!-- Ignition Gazebo Sensors Plugin (required to activate sensors) -->
+    <!--
+        Ignition Gazebo Sensors System — REQUIRED to activate any sensor.
+        Short-name form for Fortress/Humble: "ignition-gazebo-sensors-system"
+        (NOT libignition-gazebo-sensors-system.so — that's the old hardcoded path form)
+    -->
     <gazebo>
-        <plugin filename="libignition-gazebo-sensors-system.so" name="ignition::gazebo::systems::Sensors">
+        <plugin filename="ignition-gazebo-sensors-system"
+                name="ignition::gazebo::systems::Sensors">
             <render_engine>ogre2</render_engine>
         </plugin>

File: description/robot_control.xacro (robot description, xacro)
@@ -1,31 +1,57 @@
 <?xml version = "1.0"?>
 <robot xmlns:xacro="http://www.ros.org/wiki/xacro">
+<!--
+  Differential Drive plugin for Ignition Gazebo 6 (Fortress) + ROS2 Humble.
+  IMPORTANT notes on names:
+    • filename="ignition-gazebo-diff-drive-system"  ← Fortress short-name (NO lib prefix, NO .so)
+    • libgz-sim-diff-drive-system.so                ← Harmonic/Iron ONLY, does NOT exist in Humble
+-->
 <gazebo>
   <plugin
-    filename="libgz-sim-diff-drive-system.so"
-    name="gz::sim::systems::DiffDrive">
-        <!--Wheel information -->
-        <left_joint>left_wheel_joint</left_joint>
-        <right_joint>right_wheel_joint</right_joint>
-        <wheel_separation>0.35</wheel_separation>
-        <wheel_radius>0.05</wheel_radius>
-        <!-- limits — kept low to prevent wheel slip and odometry drift -->
-        <max_wheel_torque>20</max_wheel_torque>
-        <max_wheel_acceleration>1.5</max_wheel_acceleration>
-        <frame_id>odom</frame_id>
-        <child_frame_id>base_link</child_frame_id>
-        <tf_topic>/tf</tf_topic>
-        <odom_topic>/odom</odom_topic>
-        <!-- outputs-->
-        <robot_base_frame>base_link</robot_base_frame>
-        <!-- topics-->
-        <topic>cmd_vel</topic>
-        <publish_odom>true</publish_odom>
-        <publish_odom_tf>true</publish_odom_tf>
-        <publish_wheel_tf>true</publish_wheel_tf>
+    filename="ignition-gazebo-diff-drive-system"
+    name="ignition::gazebo::systems::DiffDrive">
+      <!-- Wheel joints (must match joint names in robot_core.xacro) -->
+      <left_joint>left_wheel_joint</left_joint>
+      <right_joint>right_wheel_joint</right_joint>
+      <!-- Physical parameters — must match the URDF geometry exactly -->
+      <wheel_separation>0.35</wheel_separation>
+      <wheel_radius>0.05</wheel_radius>
+      <!-- Conservative limits: prevents wheel slip which ruins odometry -->
+      <max_wheel_torque>20</max_wheel_torque>
+      <max_wheel_acceleration>1.5</max_wheel_acceleration>
+      <!-- TF frame IDs — must match SLAM/URDF frame names -->
+      <frame_id>odom</frame_id>
+      <child_frame_id>base_link</child_frame_id>
+      <!--
+        Topic — use ABSOLUTE path (leading slash) so it matches the
+        ros_gz_bridge entry exactly:  /cmd_vel@Twist]ignition.msgs.Twist
+        If you use a relative name like "cmd_vel", Ignition may namespace it
+        under the model and the bridge will never deliver commands → no motion.
+      -->
+      <topic>/cmd_vel</topic>
+      <tf_topic>/tf</tf_topic>
+      <odom_topic>/odom</odom_topic>
+      <robot_base_frame>base_link</robot_base_frame>
+      <!-- Publishing -->
+      <publish_odom>true</publish_odom>
+      <!-- odom→base_link TF published via Ignition /tf topic → bridged to ROS -->
+      <publish_odom_tf>true</publish_odom_tf>
+      <!--
+        publish_wheel_tf: publishes base_link→left_wheel / base_link→right_wheel
+        via Ignition /tf (bridged to ROS).  This lets robot_state_publisher
+        skip the wheel joint TF so we do NOT need the joint_states bridge.
+      -->
+      <publish_wheel_tf>true</publish_wheel_tf>
   </plugin>
 </gazebo>
+<!--
+  Caster wheel friction.
+  In Ignition Gazebo URDF extensions (sdformat_urdf / gz_urdf for Fortress),
+  the correct format inside <gazebo reference="..."> IS the simple element form:
+    <mu1>value</mu1>   (not <mu1 value="..."/>)
+  Keep values very low so the caster slides freely and the robot can turn.
+  The <surface><friction><ode> block does NOT work through URDF→SDF conversion.
+-->
 <gazebo reference="caster_wheel">
-  <!-- Near-zero friction so caster spins freely without resisting motion -->
   <mu1>0.001</mu1>
   <mu2>0.001</mu2>
