Commit message: fix scan riding robot + nav2 driving away: laser_yaw 180deg, disable IMU vYaw pending sign check, looser scan-match thresholds, rotate-to-heading

File: description/lidar.xacro (robot description, xacro)
@@ -13,4 +13,9 @@
   <xacro:property name="laser_y"      value="0.0"/>  <!-- left/right    -->
   <xacro:property name="laser_z"      value="0.129"/>  <!-- height above base_link (e.g. 2nd floor height) -->
+  <!-- Slamtec 0° is usually opposite the cable. If cable faces the robot rear,
+       laser +X is ~180° from base_link +X → scan rides the bot, map→odom freezes
+       while driving, and Nav2 goals look inverted vs the room. Set 0.0 if your
+       S2E 0° mark already faces the chassis front. -->
+  <xacro:property name="laser_yaw"    value="${pi}"/>
   <!-- Lidar cylinder dimensions (default ~RPLidar A1) -->
   <xacro:property name="laser_radius" value="0.035"/> <!-- 70 mm diameter -->
@@ -22,5 +27,5 @@
     <parent link="base_link"/>
     <child  link="laser_frame"/>
-    <origin xyz="${laser_x} ${laser_y} ${laser_z}" rpy="0 0 0"/>
+    <origin xyz="${laser_x} ${laser_y} ${laser_z}" rpy="0 0 ${laser_yaw}"/>
   </joint>
   <link name="laser_frame">

Commit message: before test

File: description/lidar.xacro (robot description, xacro)
@@ -14,6 +14,6 @@
        ======================================================================= -->
   <!-- LiDAR position relative to base_link  (FILL IN) -->
-  <xacro:property name="laser_x"      value="0.0"/>          <!-- chassis centre — adjust to physical mount X -->
-  <xacro:property name="laser_y"      value="0.0"/>          <!-- chassis centre — adjust to physical mount Y -->
+  <xacro:property name="laser_x"      value="-0.36"/>        <!-- 36 cm rear of chassis bottom-centre (measured) -->
+  <xacro:property name="laser_y"      value="-0.02"/>        <!-- 2 cm right of chassis centre (measured) -->
   <xacro:property name="laser_z"      value="0.10"/>         <!-- = chassis_height: LiDAR sits on top of the chassis box -->
   <!-- LiDAR yaw rotation  (FILL IN — see note above) -->
