Commit message: changed to jazzy before test

File: description/camera.xacro (robot description, xacro)
@@ -30,25 +30,3 @@
   </joint>
   <link name="camera_link_optical"/>
- <gazebo reference="camera_link">
-  <sensor name="camera" type="camera">
-      <pose>0 0 0 0 0 0</pose>
-      <topic>camera/image_raw</topic>                        <!-- NO slashes in topic name -->
-      <ignition_frame_id>camera_link_optical</ignition_frame_id>
-      <update_rate>15</update_rate>
-      <visualize>true</visualize>
-      <always_on>true</always_on>
-      <camera>
-        <horizontal_fov>1.089</horizontal_fov>           <!-- ~62 degrees -->
-        <image>
-          <format>R8G8B8</format>
-          <width>640</width>
-          <height>480</height>
-        </image>
-        <clip>
-          <near>0.05</near>
-          <far>8.0</far>
-        </clip>
-      </camera>
-    </sensor>
-  </gazebo>
 </robot>

File: description/imu.xacro (robot description, xacro)
@@ -20,16 +20,8 @@
   </collision>
 </link>
-<joint name="Rigid 5" type="fixed">
+<joint name="rigid_5" type="fixed">
   <origin xyz="-0.001839 0.002589 0.104922" rpy="0 0 0"/>
   <parent link="base_link"/>
   <child link="imu_for_urdf_1"/>
 </joint>
-<gazebo reference="imu_for_urdf_1">
-  <sensor name="imu_sensor" type="imu">
-    <always_on>1</always_on>
-    <update_rate>50</update_rate>
-    <visualize>true</visualize>
-    <topic>imu</topic>
-  </sensor>
-</gazebo>
 </robot>

File: description/lidar.xacro (robot description, xacro)
@@ -33,36 +33,3 @@
         </collision>
     </link>
-    <!-- Gazebo Lidar Color -->
-    <!-- Ignition Gazebo Lidar Plugin (GPU Lidar sensor) -->
-    <gazebo reference="laser_frame">
-        <sensor name="gpu_lidar" type="gpu_lidar">
-            <pose>0 0 0 0 0 0</pose>
-            <topic>scan</topic>
-            <ignition_frame_id>laser_frame</ignition_frame_id>
-            <update_rate>15</update_rate>
-            <visualize>true</visualize>
-            <always_on>true</always_on>
-            <ray>
-                <scan>
-                    <horizontal>
-                        <samples>360</samples>
-                        <resolution>1</resolution>
-                        <min_angle>-3.14159</min_angle>
-                        <max_angle>3.14159</max_angle>
-                    </horizontal>
-                </scan>
-                <range>
-                    <min>0.3</min>
-                    <max>12.0</max>
-                    <resolution>0.01</resolution>
-                </range>
-                <noise>
-                    <type>gaussian</type>
-                    <mean>0.0</mean>
-                    <stddev>0.01</stddev>
-                </noise>
-            </ray>
-        </sensor>
-    </gazebo>
-    <!-- Ignition Gazebo Sensors Plugin (required to activate sensors) -->
 </robot>

File: description/robot.urdf.xacro (robot description, xacro)
@@ -2,5 +2,4 @@
 <robot xmlns:xacro="http://www.ros.org/wiki/xacro"  name="robot">
   <xacro:include filename="$(find-pkg-share Ros_lidar_bot)/description/slam.xacro"/>
-  <xacro:include filename="$(find-pkg-share Ros_lidar_bot)/description/robot_control.xacro"/>
   <xacro:include filename="$(find-pkg-share Ros_lidar_bot)/description/lidar.xacro"/>
   <xacro:include filename="$(find-pkg-share Ros_lidar_bot)/description/camera.xacro"/>

File: description/slam.xacro (robot description, xacro)
@@ -1,5 +1,4 @@
 <?xml version="1.0" ?>
 <robot name="slam" xmlns:xacro="http://www.ros.org/wiki/xacro">
-<xacro:include filename="$(find-pkg-share Ros_lidar_bot)/description/slam.gazebo" />
 <link name="base_link">
   <inertial>
@@ -125,10 +124,10 @@
   <axis xyz="0.0 1.0 -0.0"/>
 </joint>
-<joint name="Rigid 3" type="fixed">
+<joint name="rigid_3" type="fixed">
   <origin xyz="-0.166839 0.002589 -0.016578" rpy="0 0 0"/>
   <parent link="base_link"/>
   <child link="ball_caster_wheel__1__1"/>
 </joint>
-<joint name="Rigid 4" type="fixed">
+<joint name="rigid_4" type="fixed">
   <origin xyz="0.163161 0.002589 -0.016578" rpy="0 0 0"/>
   <parent link="base_link"/>

Commit message: update primitive xacro geometry and teleop on device-amey

File: description/camera.xacro (robot description, xacro)
@@ -1,18 +1,36 @@
-<?xml version="1.0"?>
+<?xml version="1.0" ?>
 <robot xmlns:xacro="http://www.ros.org/wiki/xacro">
-<joint name="camera_joint" type="fixed">
+  <!-- ============================================================
+       CAMERA POSITION — FILL IN YOUR VALUES (metres, from base_link)
+       ============================================================ -->
+  <xacro:property name="cam_x"  value="0.0"/>  <!-- forward/back  -->
+  <xacro:property name="cam_y"  value="0.0"/>  <!-- left/right    -->
+  <xacro:property name="cam_z"  value="0.0"/>  <!-- height        -->
+  <!-- Camera box size  -->
+  <xacro:property name="cam_size_x" value="0.025"/>  <!-- depth         -->
+  <xacro:property name="cam_size_y" value="0.090"/>  <!-- width         -->
+  <xacro:property name="cam_size_z" value="0.025"/>  <!-- height        -->
+  <!-- ============================================================
+       CAMERA JOINT & LINK
+       ============================================================ -->
+  <joint name="camera_joint" type="fixed">
     <parent link="base_link"/>
-    <child link="camera_link"/>
-    <origin xyz="0.082 0 0.25" rpy="0 0 0"/>
+    <child  link="camera_link"/>
+    <origin xyz="${cam_x} ${cam_y} ${cam_z}" rpy="0 0 0"/>
   </joint>
   <link name="camera_link">
     <visual>
+      <origin xyz="0 0 0" rpy="0 0 0"/>
       <geometry>
-        <box size="0.010 0.03 0.03"/>
+        <box size="${cam_size_x} ${cam_size_y} ${cam_size_z}"/>
       </geometry>
+      <material name="blue">
+        <color rgba="0.0 0.3 0.8 1.0"/>
+      </material>
     </visual>
     <collision>
+      <origin xyz="0 0 0" rpy="0 0 0"/>
       <geometry>
-        <box size="0.010 0.03 0.03"/>
+        <box size="${cam_size_x} ${cam_size_y} ${cam_size_z}"/>
       </geometry>
     </collision>
@@ -20,35 +38,17 @@
       <origin xyz="0 0 0" rpy="0 0 0"/>
       <mass value="0.01"/>
-      <inertia ixx="0.0001" ixy="0" ixz="0"
-               iyy="0.0001" iyz="0" izz="0.0001"/>
+      <inertia
+        ixx="${(1.0/12.0)*0.01*(cam_size_y*cam_size_y + cam_size_z*cam_size_z)}"
+        iyy="${(1.0/12.0)*0.01*(cam_size_x*cam_size_x + cam_size_z*cam_size_z)}"
+        izz="${(1.0/12.0)*0.01*(cam_size_x*cam_size_x + cam_size_y*cam_size_y)}"
+        ixy="0" iyz="0" ixz="0"/>
     </inertial>
   </link>
+  <!-- Camera optical frame (ROS convention: Z forward, X right, Y down) -->
   <joint name="camera_optical_joint" type="fixed">
     <parent link="camera_link"/>
-    <child link="camera_link_optical"/>
-    <origin xyz="0.03 0 0" rpy="${-pi/2} 0 ${-pi/2}"/>
+    <child  link="camera_link_optical"/>
+    <origin xyz="0 0 0" rpy="${-pi/2} 0 ${-pi/2}"/>
   </joint>
   <link name="camera_link_optical"/>
- <gazebo reference="camera_link">
-  <sensor name="camera" type="camera">
-      <pose>0 0 0 0 0 0</pose>
-      <topic>camera/image_raw</topic>                        <!-- NO slashes in topic name -->
-      <ignition_frame_id>camera_link_optical</ignition_frame_id>
-      <update_rate>15</update_rate>
-      <visualize>true</visualize>
-      <always_on>true</always_on>
-      <camera>
-        <horizontal_fov>1.089</horizontal_fov>           <!-- ~62 degrees -->
-        <image>
-          <format>R8G8B8</format>
-          <width>640</width>
-          <height>480</height>
-        </image>
-        <clip>
-          <near>0.05</near>
-          <far>8.0</far>
-        </clip>
-      </camera>
-    </sensor>
-  </gazebo>
 </robot>

File: description/imu.xacro (robot description, xacro)
@@ -1,35 +1,47 @@
-<?xml version="1.0"?>
+<?xml version="1.0" ?>
 <robot xmlns:xacro="http://www.ros.org/wiki/xacro">
-<link name="imu_for_urdf_1">
-  <inertial>
-    <origin xyz="-2.395242713676784e-05 -4.697533164545013e-05 0.0011097424638633197" rpy="0 0 0"/>
-    <mass value="0.007271179941885703"/>
-    <inertia ixx="0.0" iyy="0.0" izz="1e-06" ixy="0.0" iyz="0.0" ixz="0.0"/>
-  </inertial>
-  <visual>
-    <origin xyz="0.001839 -0.002589 -0.104922" rpy="0 0 0"/>
-    <geometry>
-      <mesh filename="file://$(find Ros_lidar_bot)/meshes/imu_for_urdf_1.stl" scale="0.001 0.001 0.001"/>
-    </geometry>
-  </visual>
-  <collision>
-    <origin xyz="0.001839 -0.002589 -0.104922" rpy="0 0 0"/>
-    <geometry>
-      <mesh filename="file://$(find Ros_lidar_bot)/meshes/imu_for_urdf_1.stl" scale="0.001 0.001 0.001"/>
-    </geometry>
-  </collision>
-</link>
-<joint name="Rigid 5" type="fixed">
-  <origin xyz="-0.001839 0.002589 0.104922" rpy="0 0 0"/>
-  <parent link="base_link"/>
-  <child link="imu_for_urdf_1"/>
-</joint>
-<gazebo reference="imu_for_urdf_1">
-  <sensor name="imu_sensor" type="imu">
-    <always_on>1</always_on>
-    <update_rate>50</update_rate>
-    <visualize>true</visualize>
-    <topic>imu</topic>
-  </sensor>
-</gazebo>
+  <!-- ============================================================
+       IMU POSITION — FILL IN YOUR VALUES (metres, from base_link)
+       ============================================================ -->
+  <xacro:property name="imu_x"  value="0.0"/>  <!-- forward/back  -->
+  <xacro:property name="imu_y"  value="0.0"/>  <!-- left/right    -->
+  <xacro:property name="imu_z"  value="0.0"/>  <!-- height        -->
+  <!-- IMU box size (small PCB) -->
+  <xacro:property name="imu_size_x" value="0.030"/>
+  <xacro:property name="imu_size_y" value="0.030"/>
+  <xacro:property name="imu_size_z" value="0.010"/>
+  <!-- ============================================================
+       IMU JOINT & LINK
+       ============================================================ -->
+  <joint name="imu_joint" type="fixed">
+    <parent link="base_link"/>
+    <child  link="imu_link"/>
+    <origin xyz="${imu_x} ${imu_y} ${imu_z}" rpy="0 0 0"/>
+  </joint>
+  <link name="imu_link">
+    <visual>
+      <origin xyz="0 0 0" rpy="0 0 0"/>
+      <geometry>
+        <box size="${imu_size_x} ${imu_size_y} ${imu_size_z}"/>
+      </geometry>
+      <material name="green">
+        <color rgba="0.0 0.8 0.0 1.0"/>
+      </material>
+    </visual>
+    <collision>
+      <origin xyz="0 0 0" rpy="0 0 0"/>
+      <geometry>
+        <box size="${imu_size_x} ${imu_size_y} ${imu_size_z}"/>
+      </geometry>
+    </collision>
+    <inertial>
+      <origin xyz="0 0 0" rpy="0 0 0"/>
+      <mass value="0.01"/>
+      <inertia
+        ixx="${(1.0/12.0)*0.01*(imu_size_y*imu_size_y + imu_size_z*imu_size_z)}"
+        iyy="${(1.0/12.0)*0.01*(imu_size_x*imu_size_x + imu_size_z*imu_size_z)}"
+        izz="${(1.0/12.0)*0.01*(imu_size_x*imu_size_x + imu_size_y*imu_size_y)}"
+        ixy="0" iyz="0" ixz="0"/>
+    </inertial>
+  </link>
 </robot>

File: description/lidar.xacro (robot description, xacro)
@@ -1,68 +1,47 @@
-<?xml version="1.0"?>
+<?xml version="1.0" ?>
 <robot xmlns:xacro="http://www.ros.org/wiki/xacro">
-    <!-- LIDAR SENSOR -->
-    <!-- Lidar Joint -->
-    <!--joint name="laser_joint" type="fixed">
-        <parent link="chassis"/>
-        <child link="laser_frame"/>
-        <origin xyz="0.1 0 0.15" rpy="0 0 0"/>
-    </joint-->
-    <joint name="laser_joint" type="fixed">
-        <origin xyz="-0.001839 0.002589 0.104922" rpy="0 0 0"/>
-        <parent link="base_link"/>
-        <child link="laser_frame"/>
-    </joint>
-    <!-- Lidar Link -->
-    <link name="laser_frame">
-        <inertial>
-            <origin xyz="-4.0015749110241736e-07 -1.6278304991717424e-08 0.04331001637559857" rpy="0 0 0"/>
-    <mass value="0.5565046796809807"/>
-    <inertia ixx="0.000186" iyy="0.000186" izz="0.000341" ixy="0.0" iyz="0.0" ixz="-0.0"/>
-        </inertial>
-        <visual>
-            <origin xyz="0.001839 -0.002589 -0.104922" rpy="0 0 0"/>
-            <geometry>
-            <mesh filename="file://$(find Ros_lidar_bot)/meshes/lidar_urdf_1.stl" scale="0.001 0.001 0.001"/>
-            </geometry>
-        </visual>
-        <collision>
-            <origin xyz="0.001839 -0.002589 -0.104922" rpy="0 0 0"/>
-            <geometry>
-            <mesh filename="file://$(find Ros_lidar_bot)/meshes/lidar_urdf_1.stl" scale="0.001 0.001 0.001"/>
-            </geometry>
-        </collision>
-    </link>
-    <!-- Gazebo Lidar Color -->
-    <!-- Ignition Gazebo Lidar Plugin (GPU Lidar sensor) -->
-    <gazebo reference="laser_frame">
-        <sensor name="gpu_lidar" type="gpu_lidar">
-            <pose>0 0 0 0 0 0</pose>
-            <topic>scan</topic>
-            <ignition_frame_id>laser_frame</ignition_frame_id>
-            <update_rate>15</update_rate>
-            <visualize>true</visualize>
-            <always_on>true</always_on>
-            <ray>
-                <scan>
-                    <horizontal>
-                        <samples>360</samples>
-                        <resolution>1</resolution>
-                        <min_angle>-3.14159</min_angle>
-                        <max_angle>3.14159</max_angle>
-                    </horizontal>
-                </scan>
-                <range>
-                    <min>0.3</min>
-                    <max>12.0</max>
-                    <resolution>0.01</resolution>
-                </range>
-                <noise>
-                    <type>gaussian</type>
-                    <mean>0.0</mean>
-                    <stddev>0.01</stddev>
-                </noise>
-            </ray>
-        </sensor>
-    </gazebo>
-    <!-- Ignition Gazebo Sensors Plugin (required to activate sensors) -->
+  <!-- ============================================================
+       LIDAR POSITION — FILL IN YOUR VALUES (metres, from base_link)
+       Lidar is on the 2nd floor of the chassis.
+       ============================================================ -->
+  <xacro:property name="laser_x"      value="0.0"/>  <!-- forward/back  -->
+  <xacro:property name="laser_y"      value="0.0"/>  <!-- left/right    -->
+  <xacro:property name="laser_z"      value="0.0"/>  <!-- height above base_link (2nd floor) -->
+  <!-- Lidar cylinder dimensions (default ~RPLidar A1) -->
+  <xacro:property name="laser_radius" value="0.035"/> <!-- 70 mm diameter -->
+  <xacro:property name="laser_height" value="0.040"/> <!-- 40 mm tall     -->
+  <!-- ============================================================
+       LIDAR JOINT & LINK
+       ============================================================ -->
+  <joint name="laser_joint" type="fixed">
+    <parent link="base_link"/>
+    <child  link="laser_frame"/>
+    <origin xyz="${laser_x} ${laser_y} ${laser_z}" rpy="0 0 0"/>
+  </joint>
+  <link name="laser_frame">
+    <visual>
+      <origin xyz="0 0 0" rpy="0 0 0"/>
+      <geometry>
+        <cylinder radius="${laser_radius}" length="${laser_height}"/>
+      </geometry>
+      <material name="black">
+        <color rgba="0.1 0.1 0.1 1.0"/>
+      </material>
+    </visual>
+    <collision>
+      <origin xyz="0 0 0" rpy="0 0 0"/>
+      <geometry>
+        <cylinder radius="${laser_radius}" length="${laser_height}"/>
+      </geometry>
+    </collision>
+    <inertial>
+      <origin xyz="0 0 0" rpy="0 0 0"/>
+      <mass value="0.2"/>
+      <inertia
+        ixx="${(1.0/12.0)*0.2*(3*laser_radius*laser_radius + laser_height*laser_height)}"
+        iyy="${(1.0/12.0)*0.2*(3*laser_radius*laser_radius + laser_height*laser_height)}"
+        izz="${(1.0/2.0)*0.2*laser_radius*laser_radius}"
+        ixy="0" iyz="0" ixz="0"/>
+    </inertial>
+  </link>
 </robot>
