Commit message: update primitive xacro geometry and teleop on device-amey

File: description/slam.xacro (robot description, xacro)
@@ -1,137 +1,214 @@
 <?xml version="1.0" ?>
 <robot name="slam" xmlns:xacro="http://www.ros.org/wiki/xacro">
-<xacro:include filename="$(find Ros_lidar_bot)/description/slam.gazebo" />
-<link name="base_link">
-  <inertial>
-    <origin xyz="-0.0019297244191736867 0.0018747496550703066 0.06995619724607677" rpy="0 0 0"/>
-    <mass value="21.04115508065235"/>
-    <inertia ixx="0.188108" iyy="0.289502" izz="0.293599" ixy="-0.000208" iyz="-0.000266" ixz="-7.4e-05"/>
-  </inertial>
-  <visual>
-    <origin xyz="0 0 0" rpy="0 0 0"/>
-    <geometry>
-      <mesh filename="file://$(find Ros_lidar_bot)/meshes/base_link.stl" scale="0.001 0.001 0.001"/>
-    </geometry>
-    <material name="white">
-      <color rgba="1.0 1.0 1.0 1.0"/>
-    </material>
-  </visual>
-  <collision>
-    <origin xyz="0 0 0" rpy="0 0 0"/>
-    <geometry>
-      <mesh filename="file://$(find Ros_lidar_bot)/meshes/base_link.stl" scale="0.001 0.001 0.001"/>
-    </geometry>
-  </collision>
-</link>
-<joint name = "base_footprint_joint" type= "fixed">
-    <parent link= "base_footprint"/>
-    <child link= "base_link"/>
-    <origin xyz = "0 0 0" rpy = "0 0 0"/>
-</joint>
-<link name = "base_footprint">
-</link>
-<link name="wheel_urdf_1">
-  <inertial>
-    <origin xyz="-4.001574910018034e-07 -0.05000001627830493 -4.836244008737944e-07" rpy="0 0 0"/>
-    <mass value="7.44298937241317"/>
-    <inertia ixx="0.013521" iyy="0.024417" izz="0.013521" ixy="-0.0" iyz="0.0" ixz="0.0"/>
-  </inertial>
-  <visual>
-    <origin xyz="0.001839 0.112411 -0.034922" rpy="0 0 0"/>
-    <geometry>
-      <mesh filename="file://$(find Ros_lidar_bot)/meshes/wheel_urdf_1.stl" scale="0.001 0.001 0.001"/>
-    </geometry>
-    <material name="black">
-      <color rgba="0.00 0.00 0.00 1.0"/>
-    </material>
-  </visual>
-  <collision>
-    <origin xyz="0.001839 0.112411 -0.034922" rpy="0 0 0"/>
-    <geometry>
-      <mesh filename="file://$(find Ros_lidar_bot)/meshes/wheel_urdf_1.stl" scale="0.001 0.001 0.001"/>
-    </geometry>
-  </collision>
-</link>
-<link name="wheel_urdf__1__1">
-  <inertial>
-    <origin xyz="-4.0015749095214694e-07 0.04999998372169512 -4.836244007905277e-07" rpy="0 0 0"/>
-    <mass value="7.44298937241317"/>
-    <inertia ixx="0.013521" iyy="0.024417" izz="0.013521" ixy="0.0" iyz="0.0" ixz="-0.0"/>
-  </inertial>
-  <visual>
-    <origin xyz="0.001839 -0.117589 -0.034922" rpy="0 0 0"/>
-    <geometry>
-      <mesh filename="file://$(find Ros_lidar_bot)/meshes/wheel_urdf__1__1.stl" scale="0.001 0.001 0.001"/>
-    </geometry>
-    <material name="black">
-      <color rgba="0.00 0.00 0.00 1.0"/>
-    </material>
-  </visual>
-  <collision>
-    <origin xyz="0.001839 -0.117589 -0.034922" rpy="0 0 0"/>
-    <geometry>
-      <mesh filename="file://$(find Ros_lidar_bot)/meshes/wheel_urdf__1__1.stl" scale="0.001 0.001 0.001"/>
-    </geometry>
-  </collision>
-</link>
-<link name="ball_caster_wheel__1__1">
-  <inertial>
-    <origin xyz="-4.001574910317274e-07 -1.6278612177851592e-08 -0.012099534835058778" rpy="0 0 0"/>
-    <mass value="0.1479113408447469"/>
-    <inertia ixx="2.2e-05" iyy="2e-05" izz="2.4e-05" ixy="0.0" iyz="0.0" ixz="-0.0"/>
-  </inertial>
-  <visual>
-    <origin xyz="0.166839 -0.002589 0.016578" rpy="0 0 0"/>
-    <geometry>
-      <mesh filename="file://$(find Ros_lidar_bot)/meshes/ball_caster_wheel__1__1.stl" scale="0.001 0.001 0.001"/>
-    </geometry>
-  </visual>
-  <collision>
-    <origin xyz="0.166839 -0.002589 0.016578" rpy="0 0 0"/>
-    <geometry>
-      <mesh filename="file://$(find Ros_lidar_bot)/meshes/ball_caster_wheel__1__1.stl" scale="0.001 0.001 0.001"/>
-    </geometry>
-  </collision>
-</link>
-<link name="ball_caster_wheel_1">
-  <inertial>
-    <origin xyz="-4.001574910039718e-07 -1.627861223596483e-08 -0.012099534835058767" rpy="0 0 0"/>
-    <mass value="0.1479113408447469"/>
-    <inertia ixx="2.2e-05" iyy="2e-05" izz="2.4e-05" ixy="0.0" iyz="0.0" ixz="-0.0"/>
-  </inertial>
-  <visual>
-    <origin xyz="-0.163161 -0.002589 0.016578" rpy="0 0 0"/>
-    <geometry>
-      <mesh filename="file://$(find Ros_lidar_bot)/meshes/ball_caster_wheel_1.stl" scale="0.001 0.001 0.001"/>
-    </geometry>
-  </visual>
-  <collision>
-    <origin xyz="-0.163161 -0.002589 0.016578" rpy="0 0 0"/>
-    <geometry>
-      <mesh filename="file://$(find Ros_lidar_bot)/meshes/ball_caster_wheel_1.stl" scale="0.001 0.001 0.001"/>
-    </geometry>
-  </collision>
-</link>
-<joint name="right_wheel_joint" type="continuous">
-  <origin xyz="-0.001839 -0.112411 0.034922" rpy="0 0 0"/>
-  <parent link="base_link"/>
-  <child link="wheel_urdf_1"/>
-  <axis xyz="0.0 1.0 0.0"/>
-</joint>
-<joint name="left_wheel_joint" type="continuous">
-  <origin xyz="-0.001839 0.117589 0.034922" rpy="0 0 0"/>
-  <parent link="base_link"/>
-  <child link="wheel_urdf__1__1"/>
-  <axis xyz="0.0 1.0 -0.0"/>
-</joint>
-<joint name="Rigid 3" type="fixed">
-  <origin xyz="-0.166839 0.002589 -0.016578" rpy="0 0 0"/>
-  <parent link="base_link"/>
-  <child link="ball_caster_wheel__1__1"/>
-</joint>
-<joint name="Rigid 4" type="fixed">
-  <origin xyz="0.163161 0.002589 -0.016578" rpy="0 0 0"/>
-  <parent link="base_link"/>
-  <child link="ball_caster_wheel_1"/>
-</joint>
+  <!-- ============================================================
+       CHASSIS & WHEEL DIMENSIONS — FILL IN YOUR VALUES (metres)
+       ============================================================ -->
+  <!-- Chassis box size -->
+  <xacro:property name="chassis_length"  value="0.0"/>   <!-- front-to-back   -->
+  <xacro:property name="chassis_width"   value="0.0"/>   <!-- left-to-right   -->
+  <xacro:property name="chassis_height"  value="0.0"/>   <!-- bottom-to-top   -->
+  <!-- Drive wheel -->
+  <xacro:property name="wheel_radius"    value="0.05035"/>   <!-- RADIUS = 50.35 mm (from sketch) -->
+  <xacro:property name="wheel_width"     value="0.0"/>       <!-- axial thickness -->
+  <!-- X position of wheel axle from robot centre (0 = at centre) -->
+  <xacro:property name="wheel_x"         value="0.0"/>
+  <!-- Half-separation: each wheel is this far from the centre in Y
+       Text said 33cm → 0.165; sketch front-face shows ~35cm → 0.175
+       CONFIRM and update this value! -->
+  <xacro:property name="wheel_half_sep"  value="0.165"/>
+  <!-- Wheel centre height above chassis bottom (base_link) = 11 mm -->
+  <xacro:property name="wheel_z"         value="0.011"/>
+  <!-- Caster wheels -->
+  <xacro:property name="caster_radius"    value="0.0"/>  <!-- ball caster radius -->
+  <xacro:property name="caster_front_x"  value="0.0"/>   <!-- front caster X     -->
+  <xacro:property name="caster_rear_x"   value="0.0"/>   <!-- rear  caster X     -->
+  <!-- ============================================================
+       DERIVED VALUE
+       base_link sits (wheel_radius - wheel_z) above the ground
+       so base_footprint → base_link offset = wheel_radius - wheel_z
+       ============================================================ -->
+  <xacro:property name="ground_to_base"  value="${wheel_radius - wheel_z}"/>
+  <!-- ============================================================
+       MATERIALS
+       ============================================================ -->
+  <material name="white"><color rgba="1.0 1.0 1.0 1.0"/></material>
+  <material name="black"><color rgba="0.1 0.1 0.1 1.0"/></material>
+  <material name="grey" ><color rgba="0.5 0.5 0.5 1.0"/></material>
+  <!-- ============================================================
+       base_footprint  (ground-plane projection, zero-size link)
+       ============================================================ -->
+  <link name="base_footprint"/>
+  <!-- base_footprint → base_link
+       base_link is at the centre of the BOTTOM FACE of the chassis box.
+       It sits (wheel_radius - wheel_z) above ground so wheels touch ground. -->
+  <joint name="base_footprint_joint" type="fixed">
+    <parent link="base_footprint"/>
+    <child  link="base_link"/>
+    <origin xyz="0 0 ${ground_to_base}" rpy="0 0 0"/>
+  </joint>
+  <!-- ============================================================
+       base_link / CHASSIS
+       Visual box offset by chassis_height/2 upward so the box
+       sits entirely above base_link (= chassis bottom face centre).
+       ============================================================ -->
+  <link name="base_link">
+    <visual>
+      <origin xyz="0 0 ${chassis_height/2}" rpy="0 0 0"/>
+      <geometry>
+        <box size="${chassis_length} ${chassis_width} ${chassis_height}"/>
+      </geometry>
+      <material name="white"/>
+    </visual>
+    <collision>
+      <origin xyz="0 0 ${chassis_height/2}" rpy="0 0 0"/>
+      <geometry>
+        <box size="${chassis_length} ${chassis_width} ${chassis_height}"/>
+      </geometry>
+    </collision>
+    <inertial>
+      <!-- Centre of mass at geometric centre of box -->
+      <origin xyz="0 0 ${chassis_height/2}" rpy="0 0 0"/>
+      <mass value="2.0"/>
+      <inertia
+        ixx="${(1.0/12.0)*2.0*(chassis_width*chassis_width + chassis_height*chassis_height)}"
+        iyy="${(1.0/12.0)*2.0*(chassis_length*chassis_length + chassis_height*chassis_height)}"
+        izz="${(1.0/12.0)*2.0*(chassis_length*chassis_length + chassis_width*chassis_width)}"
+        ixy="0" iyz="0" ixz="0"/>
+    </inertial>
+  </link>
+  <!-- ============================================================
+       LEFT WHEEL  (positive Y side)
+       Joint origin = physical centre of wheel relative to base_link.
+       Link visual/collision has ZERO local offset → correct TF.
+       Cylinder lies along Z by default; rotate pi/2 about X to align
+       rotation axis with Y-axis.
+       ============================================================ -->
+  <joint name="left_wheel_joint" type="continuous">
+    <parent link="base_link"/>
+    <child  link="left_wheel"/>
+    <origin xyz="${wheel_x} ${wheel_half_sep} ${wheel_z}" rpy="0 0 0"/>
+    <axis xyz="0 1 0"/>
+  </joint>
+  <link name="left_wheel">
+    <visual>
+      <origin xyz="0 0 0" rpy="${pi/2} 0 0"/>
+      <geometry>
+        <cylinder radius="${wheel_radius}" length="${wheel_width}"/>
+      </geometry>
+      <material name="black"/>
+    </visual>
+    <collision>
+      <origin xyz="0 0 0" rpy="${pi/2} 0 0"/>
+      <geometry>
+        <cylinder radius="${wheel_radius}" length="${wheel_width}"/>
+      </geometry>
+    </collision>
+    <inertial>
+      <origin xyz="0 0 0" rpy="${pi/2} 0 0"/>
+      <mass value="0.5"/>
+      <inertia
+        ixx="${(1.0/12.0)*0.5*(3*wheel_radius*wheel_radius + wheel_width*wheel_width)}"
+        iyy="${(1.0/2.0)*0.5*wheel_radius*wheel_radius}"
+        izz="${(1.0/12.0)*0.5*(3*wheel_radius*wheel_radius + wheel_width*wheel_width)}"
+        ixy="0" iyz="0" ixz="0"/>
+    </inertial>
+  </link>
+  <!-- ============================================================
+       RIGHT WHEEL  (negative Y side)
+       ============================================================ -->
+  <joint name="right_wheel_joint" type="continuous">
+    <parent link="base_link"/>
+    <child  link="right_wheel"/>
+    <origin xyz="${wheel_x} ${-wheel_half_sep} ${wheel_z}" rpy="0 0 0"/>
+    <axis xyz="0 1 0"/>
+  </joint>
+  <link name="right_wheel">
+    <visual>
+      <origin xyz="0 0 0" rpy="${pi/2} 0 0"/>
+      <geometry>
+        <cylinder radius="${wheel_radius}" length="${wheel_width}"/>
+      </geometry>
+      <material name="black"/>
+    </visual>
+    <collision>
+      <origin xyz="0 0 0" rpy="${pi/2} 0 0"/>
+      <geometry>
+        <cylinder radius="${wheel_radius}" length="${wheel_width}"/>
+      </geometry>
+    </collision>
+    <inertial>
+      <origin xyz="0 0 0" rpy="${pi/2} 0 0"/>
+      <mass value="0.5"/>
+      <inertia
+        ixx="${(1.0/12.0)*0.5*(3*wheel_radius*wheel_radius + wheel_width*wheel_width)}"
+        iyy="${(1.0/2.0)*0.5*wheel_radius*wheel_radius}"
+        izz="${(1.0/12.0)*0.5*(3*wheel_radius*wheel_radius + wheel_width*wheel_width)}"
+        ixy="0" iyz="0" ixz="0"/>
+    </inertial>
+  </link>
+  <!-- ============================================================
+       FRONT CASTER  (passive ball caster — fixed joint)
+       ============================================================ -->
+  <joint name="caster_front_joint" type="fixed">
+    <parent link="base_link"/>
+    <child  link="caster_front_link"/>
+    <!-- caster centre sits at wheel ground level; same Z as drive wheel bottom -->
+    <origin xyz="${caster_front_x} 0 ${caster_radius}" rpy="0 0 0"/>
+  </joint>
+  <link name="caster_front_link">
+    <visual>
+      <origin xyz="0 0 0" rpy="0 0 0"/>
+      <geometry>
+        <sphere radius="${caster_radius}"/>
+      </geometry>
+      <material name="grey"/>
+    </visual>
+    <collision>
+      <origin xyz="0 0 0" rpy="0 0 0"/>
+      <geometry>
+        <sphere radius="${caster_radius}"/>
+      </geometry>
+    </collision>
+    <inertial>
+      <origin xyz="0 0 0" rpy="0 0 0"/>
+      <mass value="0.05"/>
+      <inertia
+        ixx="${(2.0/5.0)*0.05*caster_radius*caster_radius}"
+        iyy="${(2.0/5.0)*0.05*caster_radius*caster_radius}"
+        izz="${(2.0/5.0)*0.05*caster_radius*caster_radius}"
+        ixy="0" iyz="0" ixz="0"/>
+    </inertial>
+  </link>
+  <!-- ============================================================
+       REAR CASTER  (passive ball caster — fixed joint)
+       ============================================================ -->
+  <joint name="caster_rear_joint" type="fixed">
+    <parent link="base_link"/>
+    <child  link="caster_rear_link"/>
+    <origin xyz="${caster_rear_x} 0 ${caster_radius}" rpy="0 0 0"/>
+  </joint>
+  <link name="caster_rear_link">
+    <visual>
+      <origin xyz="0 0 0" rpy="0 0 0"/>
+      <geometry>
+        <sphere radius="${caster_radius}"/>
+      </geometry>
+      <material name="grey"/>
+    </visual>
+    <collision>
+      <origin xyz="0 0 0" rpy="0 0 0"/>
+      <geometry>
+        <sphere radius="${caster_radius}"/>
+      </geometry>
+    </collision>
+    <inertial>
+      <origin xyz="0 0 0" rpy="0 0 0"/>
+      <mass value="0.05"/>
+      <inertia
+        ixx="${(2.0/5.0)*0.05*caster_radius*caster_radius}"
+        iyy="${(2.0/5.0)*0.05*caster_radius*caster_radius}"
+        izz="${(2.0/5.0)*0.05*caster_radius*caster_radius}"
+        ixy="0" iyz="0" ixz="0"/>
+    </inertial>
+  </link>
 </robot>

Commit message: set realistic default dimensions and sensor offsets to prevent Gazebo DART crash

File: description/camera.xacro (robot description, xacro)
@@ -4,7 +4,7 @@
        CAMERA POSITION — FILL IN YOUR VALUES (metres, from base_link)
        ============================================================ -->
-  <xacro:property name="cam_x"  value="0.0"/>  <!-- forward/back  -->
+  <xacro:property name="cam_x"  value="0.15"/>  <!-- forward/back  -->
   <xacro:property name="cam_y"  value="0.0"/>  <!-- left/right    -->
-  <xacro:property name="cam_z"  value="0.0"/>  <!-- height        -->
+  <xacro:property name="cam_z"  value="0.10"/>  <!-- height        -->
   <!-- Camera box size  -->
   <xacro:property name="cam_size_x" value="0.025"/>  <!-- depth         -->

File: description/imu.xacro (robot description, xacro)
@@ -6,5 +6,5 @@
   <xacro:property name="imu_x"  value="0.0"/>  <!-- forward/back  -->
   <xacro:property name="imu_y"  value="0.0"/>  <!-- left/right    -->
-  <xacro:property name="imu_z"  value="0.0"/>  <!-- height        -->
+  <xacro:property name="imu_z"  value="0.05"/>  <!-- height        -->
   <!-- IMU box size (small PCB) -->
   <xacro:property name="imu_size_x" value="0.030"/>

File: description/lidar.xacro (robot description, xacro)
@@ -7,5 +7,5 @@
   <xacro:property name="laser_x"      value="0.0"/>  <!-- forward/back  -->
   <xacro:property name="laser_y"      value="0.0"/>  <!-- left/right    -->
-  <xacro:property name="laser_z"      value="0.0"/>  <!-- height above base_link (2nd floor) -->
+  <xacro:property name="laser_z"      value="0.20"/>  <!-- height above base_link (2nd floor) -->
   <!-- Lidar cylinder dimensions (default ~RPLidar A1) -->
   <xacro:property name="laser_radius" value="0.035"/> <!-- 70 mm diameter -->

File: description/slam.xacro (robot description, xacro)
@@ -5,10 +5,10 @@
        ============================================================ -->
   <!-- Chassis box size -->
-  <xacro:property name="chassis_length"  value="0.0"/>   <!-- front-to-back   -->
-  <xacro:property name="chassis_width"   value="0.0"/>   <!-- left-to-right   -->
-  <xacro:property name="chassis_height"  value="0.0"/>   <!-- bottom-to-top   -->
+  <xacro:property name="chassis_length"  value="0.33"/>   <!-- front-to-back   -->
+  <xacro:property name="chassis_width"   value="0.25"/>   <!-- left-to-right   -->
+  <xacro:property name="chassis_height"  value="0.25"/>   <!-- bottom-to-top   -->
   <!-- Drive wheel -->
   <xacro:property name="wheel_radius"    value="0.05035"/>   <!-- RADIUS = 50.35 mm (from sketch) -->
-  <xacro:property name="wheel_width"     value="0.0"/>       <!-- axial thickness -->
+  <xacro:property name="wheel_width"     value="0.04"/>       <!-- axial thickness -->
   <!-- X position of wheel axle from robot centre (0 = at centre) -->
   <xacro:property name="wheel_x"         value="0.0"/>
@@ -20,7 +20,7 @@
   <xacro:property name="wheel_z"         value="0.011"/>
   <!-- Caster wheels -->
-  <xacro:property name="caster_radius"    value="0.0"/>  <!-- ball caster radius -->
-  <xacro:property name="caster_front_x"  value="0.0"/>   <!-- front caster X     -->
-  <xacro:property name="caster_rear_x"   value="0.0"/>   <!-- rear  caster X     -->
+  <xacro:property name="caster_radius"    value="0.011"/>  <!-- ball caster radius -->
+  <xacro:property name="caster_front_x"  value="0.12"/>   <!-- front caster X     -->
+  <xacro:property name="caster_rear_x"   value="-0.12"/>   <!-- rear  caster X     -->
   <!-- ============================================================
        DERIVED VALUE
