Commit message: fix caster offsets & reset default sensor positions with offsets reference guide

File: description/camera.xacro (robot description, xacro)
@@ -1,10 +1,16 @@
 <?xml version="1.0" ?>
 <robot xmlns:xacro="http://www.ros.org/wiki/xacro">
-  <!-- ============================================================
-       CAMERA POSITION — FILL IN YOUR VALUES (metres, from base_link)
-       ============================================================ -->
-  <xacro:property name="cam_x"  value="0.15"/>  <!-- forward/back  -->
+  <!-- =======================================================================
+       CAMERA POSITION — FILL IN YOUR VALUES (metres)
+       Reference Point:
+         Measure X, Y, Z offsets relative to the 'base_link' origin.
+         - 'base_link' is located at the center of the bottom face of the chassis box.
+         - X: distance forward from the center of the chassis bottom (positive front, negative back).
+         - Y: distance left from the center of the chassis bottom (positive left, negative right).
+         - Z: height upwards from the center of the chassis bottom face.
+       ======================================================================= -->
+  <xacro:property name="cam_x"  value="0.0"/>  <!-- forward/back  -->
   <xacro:property name="cam_y"  value="0.0"/>  <!-- left/right    -->
-  <xacro:property name="cam_z"  value="0.10"/>  <!-- height        -->
+  <xacro:property name="cam_z"  value="0.0"/>  <!-- height        -->
   <!-- Camera box size  -->
   <xacro:property name="cam_size_x" value="0.025"/>  <!-- depth         -->

File: description/imu.xacro (robot description, xacro)
@@ -1,10 +1,16 @@
 <?xml version="1.0" ?>
 <robot xmlns:xacro="http://www.ros.org/wiki/xacro">
-  <!-- ============================================================
-       IMU POSITION — FILL IN YOUR VALUES (metres, from base_link)
-       ============================================================ -->
+  <!-- =======================================================================
+       IMU POSITION — FILL IN YOUR VALUES (metres)
+       Reference Point:
+         Measure X, Y, Z offsets relative to the 'base_link' origin.
+         - 'base_link' is located at the center of the bottom face of the chassis box.
+         - X: distance forward from the center of the chassis bottom (positive front, negative back).
+         - Y: distance left from the center of the chassis bottom (positive left, negative right).
+         - Z: height upwards from the center of the chassis bottom face.
+       ======================================================================= -->
   <xacro:property name="imu_x"  value="0.0"/>  <!-- forward/back  -->
   <xacro:property name="imu_y"  value="0.0"/>  <!-- left/right    -->
-  <xacro:property name="imu_z"  value="0.05"/>  <!-- height        -->
+  <xacro:property name="imu_z"  value="0.0"/>  <!-- height        -->
   <!-- IMU box size (small PCB) -->
   <xacro:property name="imu_size_x" value="0.030"/>

File: description/lidar.xacro (robot description, xacro)
@@ -1,11 +1,16 @@
 <?xml version="1.0" ?>
 <robot xmlns:xacro="http://www.ros.org/wiki/xacro">
-  <!-- ============================================================
-       LIDAR POSITION — FILL IN YOUR VALUES (metres, from base_link)
-       Lidar is on the 2nd floor of the chassis.
-       ============================================================ -->
+  <!-- =======================================================================
+       LIDAR POSITION — FILL IN YOUR VALUES (metres)
+       Reference Point:
+         Measure X, Y, Z offsets relative to the 'base_link' origin.
+         - 'base_link' is located at the center of the bottom face of the chassis box.
+         - X: distance forward from the center of the chassis bottom (positive front, negative back).
+         - Y: distance left from the center of the chassis bottom (positive left, negative right).
+         - Z: height upwards from the center of the chassis bottom face.
+       ======================================================================= -->
   <xacro:property name="laser_x"      value="0.0"/>  <!-- forward/back  -->
   <xacro:property name="laser_y"      value="0.0"/>  <!-- left/right    -->
-  <xacro:property name="laser_z"      value="0.20"/>  <!-- height above base_link (2nd floor) -->
+  <xacro:property name="laser_z"      value="0.0"/>  <!-- height above base_link (e.g. 2nd floor height) -->
   <!-- Lidar cylinder dimensions (default ~RPLidar A1) -->
   <xacro:property name="laser_radius" value="0.035"/> <!-- 70 mm diameter -->

File: description/slam.xacro (robot description, xacro)
@@ -20,5 +20,5 @@
   <xacro:property name="wheel_z"         value="0.011"/>
   <!-- Caster wheels -->
-  <xacro:property name="caster_radius"    value="0.011"/>  <!-- ball caster radius -->
+  <xacro:property name="caster_radius"    value="0.019675"/>  <!-- ball caster radius (diameter = 39.35 mm = 50.35 - 11) -->
   <xacro:property name="caster_front_x"  value="0.12"/>   <!-- front caster X     -->
   <xacro:property name="caster_rear_x"   value="-0.12"/>   <!-- rear  caster X     -->
@@ -154,5 +154,5 @@
     <child  link="caster_front_link"/>
     <!-- caster centre sits at wheel ground level; same Z as drive wheel bottom -->
-    <origin xyz="${caster_front_x} 0 ${caster_radius}" rpy="0 0 0"/>
+    <origin xyz="${caster_front_x} 0 ${-caster_radius}" rpy="0 0 0"/>
   </joint>
   <link name="caster_front_link">
@@ -186,5 +186,5 @@
     <parent link="base_link"/>
     <child  link="caster_rear_link"/>
-    <origin xyz="${caster_rear_x} 0 ${caster_radius}" rpy="0 0 0"/>
+    <origin xyz="${caster_rear_x} 0 ${-caster_radius}" rpy="0 0 0"/>
   </joint>
   <link name="caster_rear_link">

Commit message: adjust caster radius/Z-offset and add sensor coordinate reference docs

File: description/camera.xacro (robot description, xacro)
@@ -1,7 +1,13 @@
 <?xml version="1.0" ?>
 <robot xmlns:xacro="http://www.ros.org/wiki/xacro">
-  <!-- ============================================================
-       CAMERA POSITION — FILL IN YOUR VALUES (metres, from base_link)
-       ============================================================ -->
+  <!-- =======================================================================
+       CAMERA POSITION — FILL IN YOUR VALUES (metres)
+       Reference Point:
+         Measure X, Y, Z offsets relative to the 'base_link' origin.
+         - 'base_link' is located at the center of the bottom face of the chassis box.
+         - X: distance forward from the center of the chassis bottom (positive front, negative back).
+         - Y: distance left from the center of the chassis bottom (positive left, negative right).
+         - Z: height upwards from the center of the chassis bottom face.
+       ======================================================================= -->
   <xacro:property name="cam_x"  value="0.0"/>  <!-- forward/back  -->
   <xacro:property name="cam_y"  value="0.0"/>  <!-- left/right    -->

File: description/imu.xacro (robot description, xacro)
@@ -1,7 +1,13 @@
 <?xml version="1.0" ?>
 <robot xmlns:xacro="http://www.ros.org/wiki/xacro">
-  <!-- ============================================================
-       IMU POSITION — FILL IN YOUR VALUES (metres, from base_link)
-       ============================================================ -->
+  <!-- =======================================================================
+       IMU POSITION — FILL IN YOUR VALUES (metres)
+       Reference Point:
+         Measure X, Y, Z offsets relative to the 'base_link' origin.
+         - 'base_link' is located at the center of the bottom face of the chassis box.
+         - X: distance forward from the center of the chassis bottom (positive front, negative back).
+         - Y: distance left from the center of the chassis bottom (positive left, negative right).
+         - Z: height upwards from the center of the chassis bottom face.
+       ======================================================================= -->
   <xacro:property name="imu_x"  value="0.0"/>  <!-- forward/back  -->
   <xacro:property name="imu_y"  value="0.0"/>  <!-- left/right    -->

File: description/lidar.xacro (robot description, xacro)
@@ -1,11 +1,16 @@
 <?xml version="1.0" ?>
 <robot xmlns:xacro="http://www.ros.org/wiki/xacro">
-  <!-- ============================================================
-       LIDAR POSITION — FILL IN YOUR VALUES (metres, from base_link)
-       Lidar is on the 2nd floor of the chassis.
-       ============================================================ -->
+  <!-- =======================================================================
+       LIDAR POSITION — FILL IN YOUR VALUES (metres)
+       Reference Point:
+         Measure X, Y, Z offsets relative to the 'base_link' origin.
+         - 'base_link' is located at the center of the bottom face of the chassis box.
+         - X: distance forward from the center of the chassis bottom (positive front, negative back).
+         - Y: distance left from the center of the chassis bottom (positive left, negative right).
+         - Z: height upwards from the center of the chassis bottom face.
+       ======================================================================= -->
   <xacro:property name="laser_x"      value="0.0"/>  <!-- forward/back  -->
   <xacro:property name="laser_y"      value="0.0"/>  <!-- left/right    -->
-  <xacro:property name="laser_z"      value="0.0"/>  <!-- height above base_link (2nd floor) -->
+  <xacro:property name="laser_z"      value="0.0"/>  <!-- height above base_link (e.g. 2nd floor height) -->
   <!-- Lidar cylinder dimensions (default ~RPLidar A1) -->
   <xacro:property name="laser_radius" value="0.035"/> <!-- 70 mm diameter -->

File: description/slam.xacro (robot description, xacro)
@@ -5,10 +5,10 @@
        ============================================================ -->
   <!-- Chassis box size -->
-  <xacro:property name="chassis_length"  value="0.0"/>   <!-- front-to-back   -->
-  <xacro:property name="chassis_width"   value="0.0"/>   <!-- left-to-right   -->
-  <xacro:property name="chassis_height"  value="0.0"/>   <!-- bottom-to-top   -->
+  <xacro:property name="chassis_length"  value="0.33"/>   <!-- front-to-back   -->
+  <xacro:property name="chassis_width"   value="0.25"/>   <!-- left-to-right   -->
+  <xacro:property name="chassis_height"  value="0.25"/>   <!-- bottom-to-top   -->
   <!-- Drive wheel -->
   <xacro:property name="wheel_radius"    value="0.05035"/>   <!-- RADIUS = 50.35 mm (from sketch) -->
-  <xacro:property name="wheel_width"     value="0.0"/>       <!-- axial thickness -->
+  <xacro:property name="wheel_width"     value="0.04"/>       <!-- axial thickness -->
   <!-- X position of wheel axle from robot centre (0 = at centre) -->
   <xacro:property name="wheel_x"         value="0.0"/>
@@ -20,7 +20,7 @@
   <xacro:property name="wheel_z"         value="0.011"/>
   <!-- Caster wheels -->
-  <xacro:property name="caster_radius"    value="0.0"/>  <!-- ball caster radius -->
-  <xacro:property name="caster_front_x"  value="0.0"/>   <!-- front caster X     -->
-  <xacro:property name="caster_rear_x"   value="0.0"/>   <!-- rear  caster X     -->
+  <xacro:property name="caster_radius"    value="0.019675"/>  <!-- ball caster radius (diameter = 39.35 mm = 50.35 - 11) -->
+  <xacro:property name="caster_front_x"  value="0.12"/>   <!-- front caster X     -->
+  <xacro:property name="caster_rear_x"   value="-0.12"/>   <!-- rear  caster X     -->
   <!-- ============================================================
        DERIVED VALUE
@@ -154,5 +154,5 @@
     <child  link="caster_front_link"/>
     <!-- caster centre sits at wheel ground level; same Z as drive wheel bottom -->
-    <origin xyz="${caster_front_x} 0 ${caster_radius}" rpy="0 0 0"/>
+    <origin xyz="${caster_front_x} 0 ${-caster_radius}" rpy="0 0 0"/>
   </joint>
   <link name="caster_front_link">
@@ -186,5 +186,5 @@
     <parent link="base_link"/>
     <child  link="caster_rear_link"/>
-    <origin xyz="${caster_rear_x} 0 ${caster_radius}" rpy="0 0 0"/>
+    <origin xyz="${caster_rear_x} 0 ${-caster_radius}" rpy="0 0 0"/>
   </joint>
   <link name="caster_rear_link">

Commit message: vision: Ubuntu libcamerify fallback + real camera mount offset
python3-picamera2 isn't packaged in stock Ubuntu (only Raspberry Pi OS /
RPi-flavored Ubuntu images), so on this robot yolo.py's auto backend falls
back to plain cv2 -- which needs libcamerify (LD_PRELOAD V4L2->libcamera
shim) to actually open a CSI-only camera. Dashboard now wraps the vision
subprocess with libcamerify automatically when it's on PATH, so the
gamepad/dashboard toggle works without the user having to remember a
manual wrapper command; no-op if picamera2 is available instead.

camera.xacro: filled in the real mount offset (22cm forward, 26cm up from
base_link) now that the camera is physically attached.

File: description/camera.xacro (robot description, xacro)
@@ -10,7 +10,7 @@
          - Z: height upwards from the center of the chassis bottom face.
        ======================================================================= -->
-  <xacro:property name="cam_x"  value="0.0"/>  <!-- forward/back  -->
-  <xacro:property name="cam_y"  value="0.0"/>  <!-- left/right    -->
-  <xacro:property name="cam_z"  value="0.0"/>  <!-- height        -->
+  <xacro:property name="cam_x"  value="0.22"/>  <!-- forward/back  -->
+  <xacro:property name="cam_y"  value="0.0"/>   <!-- left/right    -->
+  <xacro:property name="cam_z"  value="0.26"/>  <!-- height        -->
   <!-- Camera box size  -->
   <xacro:property name="cam_size_x" value="0.025"/>  <!-- depth         -->

Commit message: camera pan/tilt head + dashboard concurrency for lower web lag
Camera (§4): new camera_servo_node drives a two-servo head — SC-15 Feetech
STS/SMS bus servo (pan, position control via scservo_sdk) and an SG90 PWM
micro servo (tilt, gpiozero). Right stick → /camera_cmd (rate control, holds
heading when centred) → servos. URDF gains pan(Z)/tilt(Y) revolute joints;
camera_servo publishes /camera_joint_states, merged by joint_state_publisher
so TF/semantics track where the camera points. Both hardware layers degrade
gracefully if the lib/device is missing. Parallel path — never touches
/cmd_vel, Nav2 or frontier exploration.

Dashboard lag (§5): run the node under a MultiThreadedExecutor with one
reentrant callback group so heavy TF/costmap ticks, sensor callbacks, the SSE
push and the nav action client no longer serialize on a single thread. Map
zlib/base64 compression moved to its own event-driven worker thread off the
ROS callback path. Nav bookkeeping guarded by a lock now that callbacks run
in parallel.

File: description/camera.xacro (robot description, xacro)
@@ -17,11 +17,41 @@
   <xacro:property name="cam_size_y" value="0.090"/>  <!-- width         -->
   <xacro:property name="cam_size_z" value="0.025"/>  <!-- height        -->
+  <!-- Servo-stack heights: base link of the SC-15 pan servo to the tilt axis,
+       and tilt axis to the camera optical centre (metres). Adjust to match the
+       manufactured mount. -->
+  <xacro:property name="pan_stack_h"  value="0.03"/>  <!-- SC-15 body height  -->
+  <xacro:property name="tilt_stack_h" value="0.03"/>  <!-- SG90 to camera     -->
+  <!-- Pan/tilt travel limits (radians) — keep in sync with camera_servo_node's
+       pan_min/max_deg and tilt_min/max_deg parameters. -->
+  <xacro:property name="pan_limit"  value="2.62"/>   <!-- ±150° -->
+  <xacro:property name="tilt_limit" value="1.40"/>   <!-- ±80°  -->
   <!-- ============================================================
-       CAMERA JOINT & LINK
+       CAMERA PAN/TILT CHAIN
+         base_link ─(fixed)─ camera_mount ─(pan, Z)─ camera_pan
+                   ─(tilt, Y)─ camera_link ─(fixed)─ camera_link_optical
        ============================================================ -->
-  <joint name="camera_joint" type="fixed">
+  <!-- Fixed mount: bottom of the SC-15 pan servo on the chassis -->
+  <joint name="camera_mount_joint" type="fixed">
     <parent link="base_link"/>
+    <child  link="camera_mount_link"/>
+    <origin xyz="${cam_x} ${cam_y} ${cam_z}" rpy="0 0 0"/>
+  </joint>
+  <link name="camera_mount_link"/>
+  <!-- PAN — SC-15 bus servo, rotates about Z -->
+  <joint name="camera_pan_joint" type="revolute">
+    <parent link="camera_mount_link"/>
+    <child  link="camera_pan_link"/>
+    <origin xyz="0 0 ${pan_stack_h}" rpy="0 0 0"/>
+    <axis xyz="0 0 1"/>
+    <limit lower="${-pan_limit}" upper="${pan_limit}" effort="20.0" velocity="6.0"/>
+  </joint>
+  <link name="camera_pan_link"/>
+  <!-- TILT — SG90 micro servo, rotates about Y -->
+  <joint name="camera_tilt_joint" type="revolute">
+    <parent link="camera_pan_link"/>
     <child  link="camera_link"/>
-    <origin xyz="${cam_x} ${cam_y} ${cam_z}" rpy="0 0 0"/>
+    <origin xyz="0 0 ${tilt_stack_h}" rpy="0 0 0"/>
+    <axis xyz="0 1 0"/>
+    <limit lower="${-tilt_limit}" upper="${tilt_limit}" effort="1.5" velocity="6.0"/>
   </joint>
   <link name="camera_link">
