Commit message: Restore Gazebo lidar/camera/imu sensors, mount sensors outside chassis, wait for Gazebo before spawning robot
Co-authored-by: Cursor <cursoragent@cursor.com>

File: description/camera.xacro (robot description, xacro)
@@ -10,7 +10,7 @@
          - Z: height upwards from the center of the chassis bottom face.
        ======================================================================= -->
-  <xacro:property name="cam_x"  value="0.0"/>  <!-- forward/back  -->
+  <xacro:property name="cam_x"  value="${chassis_length/2 + 0.0125}"/>  <!-- default: on front face (must be outside chassis) -->
   <xacro:property name="cam_y"  value="0.0"/>  <!-- left/right    -->
-  <xacro:property name="cam_z"  value="0.0"/>  <!-- height        -->
+  <xacro:property name="cam_z"  value="${chassis_height*0.6}"/>  <!-- height        -->
   <!-- Camera box size  -->
   <xacro:property name="cam_size_x" value="0.025"/>  <!-- depth         -->
@@ -58,3 +58,26 @@
   </joint>
   <link name="camera_link_optical"/>
+  <!-- Gazebo camera -> Gazebo topics camera/image_raw + camera/camera_info -->
+  <gazebo reference="camera_link">
+    <sensor name="camera" type="camera">
+      <pose>0 0 0 0 0 0</pose>
+      <topic>camera/image_raw</topic>
+      <ignition_frame_id>camera_link_optical</ignition_frame_id>
+      <update_rate>15</update_rate>
+      <visualize>true</visualize>
+      <always_on>true</always_on>
+      <camera>
+        <horizontal_fov>1.089</horizontal_fov>
+        <image>
+          <format>R8G8B8</format>
+          <width>640</width>
+          <height>480</height>
+        </image>
+        <clip>
+          <near>0.05</near>
+          <far>8.0</far>
+        </clip>
+      </camera>
+    </sensor>
+  </gazebo>
 </robot>

File: description/imu.xacro (robot description, xacro)
@@ -51,3 +51,13 @@
     </inertial>
   </link>
+  <!-- Gazebo IMU -> Gazebo topic "imu" (bridged to ROS /imu) -->
+  <gazebo reference="imu_link">
+    <sensor name="imu_sensor" type="imu">
+      <always_on>1</always_on>
+      <update_rate>50</update_rate>
+      <visualize>true</visualize>
+      <topic>imu</topic>
+      <ignition_frame_id>imu_link</ignition_frame_id>
+    </sensor>
+  </gazebo>
 </robot>

File: description/lidar.xacro (robot description, xacro)
@@ -12,8 +12,10 @@
   <xacro:property name="laser_x"      value="0.0"/>  <!-- forward/back  -->
   <xacro:property name="laser_y"      value="0.0"/>  <!-- left/right    -->
-  <xacro:property name="laser_z"      value="0.0"/>  <!-- height above base_link (e.g. 2nd floor height) -->
   <!-- Lidar cylinder dimensions (default ~RPLidar A1) -->
   <xacro:property name="laser_radius" value="0.035"/> <!-- 70 mm diameter -->
   <xacro:property name="laser_height" value="0.040"/> <!-- 40 mm tall     -->
+  <!-- Default: mounted ON TOP of the chassis. Must be above the chassis top
+       (chassis_height) or the chassis blocks every ray and /scan is empty. -->
+  <xacro:property name="laser_z"      value="${chassis_height + laser_height/2}"/>
   <!-- ============================================================
        LIDAR JOINT & LINK
@@ -50,3 +52,34 @@
     </inertial>
   </link>
+  <!-- Gazebo GPU lidar -> Gazebo topic "scan" (bridged to ROS /scan) -->
+  <gazebo reference="laser_frame">
+    <sensor name="gpu_lidar" type="gpu_lidar">
+      <pose>0 0 0 0 0 0</pose>
+      <topic>scan</topic>
+      <ignition_frame_id>laser_frame</ignition_frame_id>
+      <update_rate>15</update_rate>
+      <visualize>true</visualize>
+      <always_on>true</always_on>
+      <ray>
+        <scan>
+          <horizontal>
+            <samples>360</samples>
+            <resolution>1</resolution>
+            <min_angle>-3.14159</min_angle>
+            <max_angle>3.14159</max_angle>
+          </horizontal>
+        </scan>
+        <range>
+          <min>0.15</min>
+          <max>12.0</max>
+          <resolution>0.01</resolution>
+        </range>
+        <noise>
+          <type>gaussian</type>
+          <mean>0.0</mean>
+          <stddev>0.01</stddev>
+        </noise>
+      </ray>
+    </sensor>
+  </gazebo>
 </robot>
