Commit message: feat: Jazzy migration + RPi5 hardware sanity fixes
ROS 2 Jazzy migration (all files):
- package.xml: add ament_cmake_ros buildtool dep
- CMakeLists.txt: C++17 standard
- config/ekf.yaml: use_sim_time false (hardware deploy)
- config/nav2_params.yaml: use_sim_time false everywhere,
  observation_keep_time (renamed from observation_persistence in Jazzy)
- config/mapper_params_*.yaml: map_update_frequency (renamed from interval)
- description/*.xacro:  throughout

Hardware sanity fixes:
- Ros_lidar_bot/driver_node.py: wheel_radius 0.033→0.081m,
  wheel_base 0.160→0.3395m (match robot_control.xacro)
- Ros_lidar_bot/odom_node.py: same wheel param corrections
- Ros_lidar_bot/lidar_node.py: frame_id default 'laser'→'laser_frame'
  (match URDF link name to fix TF lookups in Nav2/SLAM)
- Ros_lidar_bot/imu_node.py: frame_id default 'imu_link'→'imu_for_urdf_1'
  (match URDF link name)
- setup.py: add missing entry_points for safety_stop_node and
  semantic_slam_node; fix frontier_explorer→frontier_explorer_node
- launch/launch_robot.launch.py: executable names use setup.py
  console_scripts keys (not .py suffix); imu frame_id updated
- launch/autonomous_robot.launch.py: frontier_explorer executable fixed

RPi5 deployment:
- install_rpi5_jazzy.sh: full setup script for Ubuntu 24.04 / ROS 2 Jazzy

File: description/imu.xacro (robot description, xacro)
@@ -10,5 +10,5 @@
     <origin xyz="0.001839 -0.002589 -0.104922" rpy="0 0 0"/>
     <geometry>
-      <mesh filename="file://$(find Ros_lidar_bot)/meshes/imu_for_urdf_1.stl" scale="0.001 0.001 0.001"/>
+      <mesh filename="file://$(find-pkg-share Ros_lidar_bot)/meshes/imu_for_urdf_1.stl" scale="0.001 0.001 0.001"/>
     </geometry>
   </visual>
@@ -16,5 +16,5 @@
     <origin xyz="0.001839 -0.002589 -0.104922" rpy="0 0 0"/>
     <geometry>
-      <mesh filename="file://$(find Ros_lidar_bot)/meshes/imu_for_urdf_1.stl" scale="0.001 0.001 0.001"/>
+      <mesh filename="file://$(find-pkg-share Ros_lidar_bot)/meshes/imu_for_urdf_1.stl" scale="0.001 0.001 0.001"/>
     </geometry>
   </collision>

File: description/lidar.xacro (robot description, xacro)
@@ -23,5 +23,5 @@
             <origin xyz="0.001839 -0.002589 -0.104922" rpy="0 0 0"/>
             <geometry>
-            <mesh filename="file://$(find Ros_lidar_bot)/meshes/lidar_urdf_1.stl" scale="0.001 0.001 0.001"/>
+            <mesh filename="file://$(find-pkg-share Ros_lidar_bot)/meshes/lidar_urdf_1.stl" scale="0.001 0.001 0.001"/>
             </geometry>
         </visual>
@@ -29,5 +29,5 @@
             <origin xyz="0.001839 -0.002589 -0.104922" rpy="0 0 0"/>
             <geometry>
-            <mesh filename="file://$(find Ros_lidar_bot)/meshes/lidar_urdf_1.stl" scale="0.001 0.001 0.001"/>
+            <mesh filename="file://$(find-pkg-share Ros_lidar_bot)/meshes/lidar_urdf_1.stl" scale="0.001 0.001 0.001"/>
             </geometry>
         </collision>

File: description/robot.urdf.xacro (robot description, xacro)
@@ -1,8 +1,8 @@
 <?xml version="1.0"?>
 <robot xmlns:xacro="http://www.ros.org/wiki/xacro"  name="robot">
-  <xacro:include filename="$(find Ros_lidar_bot)/description/slam.xacro"/>
-  <xacro:include filename="$(find Ros_lidar_bot)/description/robot_control.xacro"/>
-  <xacro:include filename="$(find Ros_lidar_bot)/description/lidar.xacro"/>
-  <xacro:include filename="$(find Ros_lidar_bot)/description/camera.xacro"/>
-  <xacro:include filename="$(find Ros_lidar_bot)/description/imu.xacro"/>
+  <xacro:include filename="$(find-pkg-share Ros_lidar_bot)/description/slam.xacro"/>
+  <xacro:include filename="$(find-pkg-share Ros_lidar_bot)/description/robot_control.xacro"/>
+  <xacro:include filename="$(find-pkg-share Ros_lidar_bot)/description/lidar.xacro"/>
+  <xacro:include filename="$(find-pkg-share Ros_lidar_bot)/description/camera.xacro"/>
+  <xacro:include filename="$(find-pkg-share Ros_lidar_bot)/description/imu.xacro"/>
 </robot>

File: description/slam.xacro (robot description, xacro)
@@ -1,5 +1,5 @@
 <?xml version="1.0" ?>
 <robot name="slam" xmlns:xacro="http://www.ros.org/wiki/xacro">
-<xacro:include filename="$(find Ros_lidar_bot)/description/slam.gazebo" />
+<xacro:include filename="$(find-pkg-share Ros_lidar_bot)/description/slam.gazebo" />
 <link name="base_link">
   <inertial>
@@ -11,5 +11,5 @@
     <origin xyz="0 0 0" rpy="0 0 0"/>
     <geometry>
-      <mesh filename="file://$(find Ros_lidar_bot)/meshes/base_link.stl" scale="0.001 0.001 0.001"/>
+      <mesh filename="file://$(find-pkg-share Ros_lidar_bot)/meshes/base_link.stl" scale="0.001 0.001 0.001"/>
     </geometry>
     <material name="white">
@@ -20,5 +20,5 @@
     <origin xyz="0 0 0" rpy="0 0 0"/>
     <geometry>
-      <mesh filename="file://$(find Ros_lidar_bot)/meshes/base_link.stl" scale="0.001 0.001 0.001"/>
+      <mesh filename="file://$(find-pkg-share Ros_lidar_bot)/meshes/base_link.stl" scale="0.001 0.001 0.001"/>
     </geometry>
   </collision>
@@ -40,5 +40,5 @@
     <origin xyz="0.001839 0.112411 -0.034922" rpy="0 0 0"/>
     <geometry>
-      <mesh filename="file://$(find Ros_lidar_bot)/meshes/wheel_urdf_1.stl" scale="0.001 0.001 0.001"/>
+      <mesh filename="file://$(find-pkg-share Ros_lidar_bot)/meshes/wheel_urdf_1.stl" scale="0.001 0.001 0.001"/>
     </geometry>
     <material name="black">
@@ -49,5 +49,5 @@
     <origin xyz="0.001839 0.112411 -0.034922" rpy="0 0 0"/>
     <geometry>
-      <mesh filename="file://$(find Ros_lidar_bot)/meshes/wheel_urdf_1.stl" scale="0.001 0.001 0.001"/>
+      <mesh filename="file://$(find-pkg-share Ros_lidar_bot)/meshes/wheel_urdf_1.stl" scale="0.001 0.001 0.001"/>
     </geometry>
   </collision>
@@ -62,5 +62,5 @@
     <origin xyz="0.001839 -0.117589 -0.034922" rpy="0 0 0"/>
     <geometry>
-      <mesh filename="file://$(find Ros_lidar_bot)/meshes/wheel_urdf__1__1.stl" scale="0.001 0.001 0.001"/>
+      <mesh filename="file://$(find-pkg-share Ros_lidar_bot)/meshes/wheel_urdf__1__1.stl" scale="0.001 0.001 0.001"/>
     </geometry>
     <material name="black">
@@ -71,5 +71,5 @@
     <origin xyz="0.001839 -0.117589 -0.034922" rpy="0 0 0"/>
     <geometry>
-      <mesh filename="file://$(find Ros_lidar_bot)/meshes/wheel_urdf__1__1.stl" scale="0.001 0.001 0.001"/>
+      <mesh filename="file://$(find-pkg-share Ros_lidar_bot)/meshes/wheel_urdf__1__1.stl" scale="0.001 0.001 0.001"/>
     </geometry>
   </collision>
@@ -84,5 +84,5 @@
     <origin xyz="0.166839 -0.002589 0.016578" rpy="0 0 0"/>
     <geometry>
-      <mesh filename="file://$(find Ros_lidar_bot)/meshes/ball_caster_wheel__1__1.stl" scale="0.001 0.001 0.001"/>
+      <mesh filename="file://$(find-pkg-share Ros_lidar_bot)/meshes/ball_caster_wheel__1__1.stl" scale="0.001 0.001 0.001"/>
     </geometry>
   </visual>
@@ -90,5 +90,5 @@
     <origin xyz="0.166839 -0.002589 0.016578" rpy="0 0 0"/>
     <geometry>
-      <mesh filename="file://$(find Ros_lidar_bot)/meshes/ball_caster_wheel__1__1.stl" scale="0.001 0.001 0.001"/>
+      <mesh filename="file://$(find-pkg-share Ros_lidar_bot)/meshes/ball_caster_wheel__1__1.stl" scale="0.001 0.001 0.001"/>
     </geometry>
   </collision>
@@ -103,5 +103,5 @@
     <origin xyz="-0.163161 -0.002589 0.016578" rpy="0 0 0"/>
     <geometry>
-      <mesh filename="file://$(find Ros_lidar_bot)/meshes/ball_caster_wheel_1.stl" scale="0.001 0.001 0.001"/>
+      <mesh filename="file://$(find-pkg-share Ros_lidar_bot)/meshes/ball_caster_wheel_1.stl" scale="0.001 0.001 0.001"/>
     </geometry>
   </visual>
@@ -109,5 +109,5 @@
     <origin xyz="-0.163161 -0.002589 0.016578" rpy="0 0 0"/>
     <geometry>
-      <mesh filename="file://$(find Ros_lidar_bot)/meshes/ball_caster_wheel_1.stl" scale="0.001 0.001 0.001"/>
+      <mesh filename="file://$(find-pkg-share Ros_lidar_bot)/meshes/ball_caster_wheel_1.stl" scale="0.001 0.001 0.001"/>
     </geometry>
   </collision>

Commit message: before testing rviz2

File: description/imu.xacro (robot description, xacro)
@@ -10,5 +10,5 @@
     <origin xyz="0.001839 -0.002589 -0.104922" rpy="0 0 0"/>
     <geometry>
-      <mesh filename="file://$(find-pkg-share Ros_lidar_bot)/meshes/imu_for_urdf_1.stl" scale="0.001 0.001 0.001"/>
+      <mesh filename="file://$(find Ros_lidar_bot)/meshes/imu_for_urdf_1.stl" scale="0.001 0.001 0.001"/>
     </geometry>
   </visual>
@@ -16,5 +16,5 @@
     <origin xyz="0.001839 -0.002589 -0.104922" rpy="0 0 0"/>
     <geometry>
-      <mesh filename="file://$(find-pkg-share Ros_lidar_bot)/meshes/imu_for_urdf_1.stl" scale="0.001 0.001 0.001"/>
+      <mesh filename="file://$(find Ros_lidar_bot)/meshes/imu_for_urdf_1.stl" scale="0.001 0.001 0.001"/>
     </geometry>
   </collision>

File: description/lidar.xacro (robot description, xacro)
@@ -23,5 +23,5 @@
             <origin xyz="0.001839 -0.002589 -0.104922" rpy="0 0 0"/>
             <geometry>
-            <mesh filename="file://$(find-pkg-share Ros_lidar_bot)/meshes/lidar_urdf_1.stl" scale="0.001 0.001 0.001"/>
+            <mesh filename="file://$(find Ros_lidar_bot)/meshes/lidar_urdf_1.stl" scale="0.001 0.001 0.001"/>
             </geometry>
         </visual>
@@ -29,5 +29,5 @@
             <origin xyz="0.001839 -0.002589 -0.104922" rpy="0 0 0"/>
             <geometry>
-            <mesh filename="file://$(find-pkg-share Ros_lidar_bot)/meshes/lidar_urdf_1.stl" scale="0.001 0.001 0.001"/>
+            <mesh filename="file://$(find Ros_lidar_bot)/meshes/lidar_urdf_1.stl" scale="0.001 0.001 0.001"/>
             </geometry>
         </collision>

File: description/robot.urdf.xacro (robot description, xacro)
@@ -1,7 +1,7 @@
 <?xml version="1.0"?>
 <robot xmlns:xacro="http://www.ros.org/wiki/xacro"  name="robot">
-  <xacro:include filename="$(find-pkg-share Ros_lidar_bot)/description/slam.xacro"/>
-  <xacro:include filename="$(find-pkg-share Ros_lidar_bot)/description/lidar.xacro"/>
-  <xacro:include filename="$(find-pkg-share Ros_lidar_bot)/description/camera.xacro"/>
-  <xacro:include filename="$(find-pkg-share Ros_lidar_bot)/description/imu.xacro"/>
+  <xacro:include filename="$(find Ros_lidar_bot)/description/slam.xacro"/>
+  <xacro:include filename="$(find Ros_lidar_bot)/description/lidar.xacro"/>
+  <xacro:include filename="$(find Ros_lidar_bot)/description/camera.xacro"/>
+  <xacro:include filename="$(find Ros_lidar_bot)/description/imu.xacro"/>
 </robot>

File: description/slam.xacro (robot description, xacro)
@@ -10,5 +10,5 @@
     <origin xyz="0 0 0" rpy="0 0 0"/>
     <geometry>
-      <mesh filename="file://$(find-pkg-share Ros_lidar_bot)/meshes/base_link.stl" scale="0.001 0.001 0.001"/>
+      <mesh filename="file://$(find Ros_lidar_bot)/meshes/base_link.stl" scale="0.001 0.001 0.001"/>
     </geometry>
     <material name="white">
@@ -19,5 +19,5 @@
     <origin xyz="0 0 0" rpy="0 0 0"/>
     <geometry>
-      <mesh filename="file://$(find-pkg-share Ros_lidar_bot)/meshes/base_link.stl" scale="0.001 0.001 0.001"/>
+      <mesh filename="file://$(find Ros_lidar_bot)/meshes/base_link.stl" scale="0.001 0.001 0.001"/>
     </geometry>
   </collision>
@@ -37,7 +37,7 @@
   </inertial>
   <visual>
-    <origin xyz="0.001839 0.112411 -0.034922" rpy="0 0 0"/>
+    <origin xyz="0.001839 0.162411 -0.034922" rpy="0 0 0"/>
     <geometry>
-      <mesh filename="file://$(find-pkg-share Ros_lidar_bot)/meshes/wheel_urdf_1.stl" scale="0.001 0.001 0.001"/>
+      <mesh filename="file://$(find Ros_lidar_bot)/meshes/wheel_urdf_1.stl" scale="0.001 0.001 0.001"/>
     </geometry>
     <material name="black">
@@ -46,7 +46,7 @@
   </visual>
   <collision>
-    <origin xyz="0.001839 0.112411 -0.034922" rpy="0 0 0"/>
+    <origin xyz="0.001839 0.162411 -0.034922" rpy="0 0 0"/>
     <geometry>
-      <mesh filename="file://$(find-pkg-share Ros_lidar_bot)/meshes/wheel_urdf_1.stl" scale="0.001 0.001 0.001"/>
+      <mesh filename="file://$(find Ros_lidar_bot)/meshes/wheel_urdf_1.stl" scale="0.001 0.001 0.001"/>
     </geometry>
   </collision>
@@ -59,7 +59,7 @@
   </inertial>
   <visual>
-    <origin xyz="0.001839 -0.117589 -0.034922" rpy="0 0 0"/>
+    <origin xyz="0.001839 -0.167589 -0.034922" rpy="0 0 0"/>
     <geometry>
-      <mesh filename="file://$(find-pkg-share Ros_lidar_bot)/meshes/wheel_urdf__1__1.stl" scale="0.001 0.001 0.001"/>
+      <mesh filename="file://$(find Ros_lidar_bot)/meshes/wheel_urdf__1__1.stl" scale="0.001 0.001 0.001"/>
     </geometry>
     <material name="black">
@@ -68,7 +68,7 @@
   </visual>
   <collision>
-    <origin xyz="0.001839 -0.117589 -0.034922" rpy="0 0 0"/>
+    <origin xyz="0.001839 -0.167589 -0.034922" rpy="0 0 0"/>
     <geometry>
-      <mesh filename="file://$(find-pkg-share Ros_lidar_bot)/meshes/wheel_urdf__1__1.stl" scale="0.001 0.001 0.001"/>
+      <mesh filename="file://$(find Ros_lidar_bot)/meshes/wheel_urdf__1__1.stl" scale="0.001 0.001 0.001"/>
     </geometry>
   </collision>
@@ -83,5 +83,5 @@
     <origin xyz="0.166839 -0.002589 0.016578" rpy="0 0 0"/>
     <geometry>
-      <mesh filename="file://$(find-pkg-share Ros_lidar_bot)/meshes/ball_caster_wheel__1__1.stl" scale="0.001 0.001 0.001"/>
+      <mesh filename="file://$(find Ros_lidar_bot)/meshes/ball_caster_wheel__1__1.stl" scale="0.001 0.001 0.001"/>
     </geometry>
   </visual>
@@ -89,5 +89,5 @@
     <origin xyz="0.166839 -0.002589 0.016578" rpy="0 0 0"/>
     <geometry>
-      <mesh filename="file://$(find-pkg-share Ros_lidar_bot)/meshes/ball_caster_wheel__1__1.stl" scale="0.001 0.001 0.001"/>
+      <mesh filename="file://$(find Ros_lidar_bot)/meshes/ball_caster_wheel__1__1.stl" scale="0.001 0.001 0.001"/>
     </geometry>
   </collision>
@@ -102,5 +102,5 @@
     <origin xyz="-0.163161 -0.002589 0.016578" rpy="0 0 0"/>
     <geometry>
-      <mesh filename="file://$(find-pkg-share Ros_lidar_bot)/meshes/ball_caster_wheel_1.stl" scale="0.001 0.001 0.001"/>
+      <mesh filename="file://$(find Ros_lidar_bot)/meshes/ball_caster_wheel_1.stl" scale="0.001 0.001 0.001"/>
     </geometry>
   </visual>
@@ -108,10 +108,10 @@
     <origin xyz="-0.163161 -0.002589 0.016578" rpy="0 0 0"/>
     <geometry>
-      <mesh filename="file://$(find-pkg-share Ros_lidar_bot)/meshes/ball_caster_wheel_1.stl" scale="0.001 0.001 0.001"/>
+      <mesh filename="file://$(find Ros_lidar_bot)/meshes/ball_caster_wheel_1.stl" scale="0.001 0.001 0.001"/>
     </geometry>
   </collision>
 </link>
 <joint name="right_wheel_joint" type="continuous">
-  <origin xyz="-0.001839 -0.112411 0.034922" rpy="0 0 0"/>
+  <origin xyz="-0.001839 -0.162411 0.034922" rpy="0 0 0"/>
   <parent link="base_link"/>
   <child link="wheel_urdf_1"/>
@@ -119,5 +119,5 @@
 </joint>
 <joint name="left_wheel_joint" type="continuous">
-  <origin xyz="-0.001839 0.117589 0.034922" rpy="0 0 0"/>
+  <origin xyz="-0.001839 0.167589 0.034922" rpy="0 0 0"/>
   <parent link="base_link"/>
   <child link="wheel_urdf__1__1"/>

Commit message: updated the location of the items before test

File: description/imu.xacro (robot description, xacro)
@@ -10,11 +10,11 @@
          - Z: height upwards from the center of the chassis bottom face.
        ======================================================================= -->
-  <xacro:property name="imu_x"  value="0.0"/>  <!-- forward/back  -->
+  <xacro:property name="imu_x"  value="-0.115"/>  <!-- forward/back  -->
   <xacro:property name="imu_y"  value="0.0"/>  <!-- left/right    -->
-  <xacro:property name="imu_z"  value="0.0"/>  <!-- height        -->
+  <xacro:property name="imu_z"  value="0.004"/>  <!-- height        -->
   <!-- IMU box size (small PCB) -->
   <xacro:property name="imu_size_x" value="0.030"/>
-  <xacro:property name="imu_size_y" value="0.030"/>
-  <xacro:property name="imu_size_z" value="0.010"/>
+  <xacro:property name="imu_size_y" value="0.020"/>
+  <xacro:property name="imu_size_z" value="0.001"/>
   <!-- ============================================================
        IMU JOINT & LINK

File: description/lidar.xacro (robot description, xacro)
@@ -12,5 +12,5 @@
   <xacro:property name="laser_x"      value="0.0"/>  <!-- forward/back  -->
   <xacro:property name="laser_y"      value="0.0"/>  <!-- left/right    -->
-  <xacro:property name="laser_z"      value="0.0"/>  <!-- height above base_link (e.g. 2nd floor height) -->
+  <xacro:property name="laser_z"      value="0.129"/>  <!-- height above base_link (e.g. 2nd floor height) -->
   <!-- Lidar cylinder dimensions (default ~RPLidar A1) -->
   <xacro:property name="laser_radius" value="0.035"/> <!-- 70 mm diameter -->

File: description/slam.xacro (robot description, xacro)
@@ -5,7 +5,7 @@
        ============================================================ -->
   <!-- Chassis box size -->
-  <xacro:property name="chassis_length"  value="0.33"/>   <!-- front-to-back   -->
+  <xacro:property name="chassis_length"  value="0.45"/>   <!-- front-to-back   -->
   <xacro:property name="chassis_width"   value="0.25"/>   <!-- left-to-right   -->
-  <xacro:property name="chassis_height"  value="0.25"/>   <!-- bottom-to-top   -->
+  <xacro:property name="chassis_height"  value="0.20"/>   <!-- bottom-to-top   -->
   <!-- Drive wheel -->
   <xacro:property name="wheel_radius"    value="0.05035"/>   <!-- RADIUS = 50.35 mm (from sketch) -->

Commit message: reverted directions of y and z axis of imu, keeping x axis same

File: description/imu.xacro (robot description, xacro)
@@ -23,5 +23,5 @@
     <parent link="base_link"/>
     <child  link="imu_link"/>
-    <origin xyz="${imu_x} ${imu_y} ${imu_z}" rpy="0 0 0"/>
+    <origin xyz="${imu_x} ${imu_y} ${imu_z}" rpy="${pi} 0 0"/>
   </joint>
   <link name="imu_link">

Commit message: updated the orientation of imu and bot's y & z axis

File: description/imu.xacro (robot description, xacro)
@@ -23,5 +23,5 @@
     <parent link="base_link"/>
     <child  link="imu_link"/>
-    <origin xyz="${imu_x} ${imu_y} ${imu_z}" rpy="${pi} 0 0"/>
+    <origin xyz="${imu_x} ${imu_y} ${imu_z}" rpy="0 0 0"/>
   </joint>
   <link name="imu_link">
