Commit message: added some nodes

File: description/imu.xacro (robot description, xacro)
@@ -3,18 +3,27 @@
   <!-- =======================================================================
        IMU POSITION — FILL IN YOUR VALUES (metres)
-       Reference Point:
-         Measure X, Y, Z offsets relative to the 'base_link' origin.
-         - 'base_link' is located at the center of the bottom face of the chassis box.
-         - X: distance forward from the center of the chassis bottom (positive front, negative back).
-         - Y: distance left from the center of the chassis bottom (positive left, negative right).
-         - Z: height upwards from the center of the chassis bottom face.
+       Reference frame:
+         'base_link' is at the centre of the BOTTOM FACE of the chassis box.
+         X : forward from chassis centre  (+front, -rear)
+         Y : left from chassis centre     (+left,  -right)
+         Z : height above chassis bottom  (upward positive)
+       How to measure:
+         1. Place the bot on a flat surface.
+         2. Find the IMU chip/PCB mounting point.
+         3. Measure its X/Y/Z offset from the chassis bottom-centre.
        ======================================================================= -->
-  <xacro:property name="imu_x"  value="-0.115"/>  <!-- forward/back  -->
-  <xacro:property name="imu_y"  value="0.0"/>  <!-- left/right    -->
-  <xacro:property name="imu_z"  value="0.004"/>  <!-- height        -->
-  <!-- IMU box size (small PCB) -->
-  <xacro:property name="imu_size_x" value="0.030"/>
-  <xacro:property name="imu_size_y" value="0.020"/>
-  <xacro:property name="imu_size_z" value="0.001"/>
+  <!-- IMU position relative to base_link  (FILL IN) -->
+  <xacro:property name="imu_x"  value="TODO_FILL"/>   <!-- e.g.  0.05  -->
+  <xacro:property name="imu_y"  value="TODO_FILL"/>   <!-- e.g.  0.0   -->
+  <xacro:property name="imu_z"  value="TODO_FILL"/>   <!-- e.g.  0.12  -->
+  <!-- IMU orientation offset (FILL IN if the IMU is not mounted flat)
+       Leave all zeros if the IMU X axis points robot-forward and Z is up. -->
+  <xacro:property name="imu_roll"  value="0.0"/>
+  <xacro:property name="imu_pitch" value="0.0"/>
+  <xacro:property name="imu_yaw"   value="0.0"/>
+  <!-- IMU PCB box size — only used for visualisation (FILL IN or leave as-is) -->
+  <xacro:property name="imu_size_x" value="0.030"/>   <!-- 30 mm long -->
+  <xacro:property name="imu_size_y" value="0.020"/>   <!-- 20 mm wide -->
+  <xacro:property name="imu_size_z" value="0.004"/>   <!--  4 mm tall -->
   <!-- ============================================================
        IMU JOINT & LINK
@@ -23,5 +32,6 @@
     <parent link="base_link"/>
     <child  link="imu_link"/>
-    <origin xyz="${imu_x} ${imu_y} ${imu_z}" rpy="0 0 0"/>
+    <origin xyz="${imu_x} ${imu_y} ${imu_z}"
+            rpy="${imu_roll} ${imu_pitch} ${imu_yaw}"/>
   </joint>
   <link name="imu_link">
@@ -43,5 +53,5 @@
     <inertial>
       <origin xyz="0 0 0" rpy="0 0 0"/>
-      <mass value="0.01"/>
+      <mass value="0.010"/>
       <inertia
         ixx="${(1.0/12.0)*0.01*(imu_size_y*imu_size_y + imu_size_z*imu_size_z)}"

File: description/lidar.xacro (robot description, xacro)
@@ -3,22 +3,23 @@
   <!-- =======================================================================
        LIDAR POSITION — FILL IN YOUR VALUES (metres)
-       Reference Point:
-         Measure X, Y, Z offsets relative to the 'base_link' origin.
-         - 'base_link' is located at the center of the bottom face of the chassis box.
-         - X: distance forward from the center of the chassis bottom (positive front, negative back).
-         - Y: distance left from the center of the chassis bottom (positive left, negative right).
-         - Z: height upwards from the center of the chassis bottom face.
+       Reference frame:
+         'base_link' is at the centre of the BOTTOM FACE of the chassis box.
+         X : forward from chassis centre  (+front, -rear)
+         Y : left from chassis centre     (+left,  -right)
+         Z : height above chassis bottom  (upward positive)
+       laser_yaw:
+         0.0  → LiDAR "0°" mark faces robot front  (most common)
+         pi   → LiDAR "0°" mark faces robot rear   (flip if scan is mirrored)
+         Measure the physical orientation of the LiDAR cable/mark on the chassis.
        ======================================================================= -->
-  <xacro:property name="laser_x"      value="0.0"/>  <!-- forward/back  -->
-  <xacro:property name="laser_y"      value="0.0"/>  <!-- left/right    -->
-  <xacro:property name="laser_z"      value="0.129"/>  <!-- height above base_link (e.g. 2nd floor height) -->
-  <!-- Slamtec 0° is usually opposite the cable. If cable faces the robot rear,
-       laser +X is ~180° from base_link +X → scan rides the bot, map→odom freezes
-       while driving, and Nav2 goals look inverted vs the room. Set 0.0 if your
-       S2E 0° mark already faces the chassis front. -->
-  <xacro:property name="laser_yaw"    value="${pi}"/>
-  <!-- Lidar cylinder dimensions (default ~RPLidar A1) -->
-  <xacro:property name="laser_radius" value="0.035"/> <!-- 70 mm diameter -->
-  <xacro:property name="laser_height" value="0.040"/> <!-- 40 mm tall     -->
+  <!-- LiDAR position relative to base_link  (FILL IN) -->
+  <xacro:property name="laser_x"      value="TODO_FILL"/>   <!-- e.g.  0.0   -->
+  <xacro:property name="laser_y"      value="TODO_FILL"/>   <!-- e.g.  0.0   -->
+  <xacro:property name="laser_z"      value="TODO_FILL"/>   <!-- e.g.  0.18  (height of LiDAR above chassis bottom) -->
+  <!-- LiDAR yaw rotation  (FILL IN — see note above) -->
+  <xacro:property name="laser_yaw"    value="TODO_FILL"/>   <!-- 0.0 or ${pi} -->
+  <!-- LiDAR cylinder visual dimensions  (FILL IN or leave defaults) -->
+  <xacro:property name="laser_radius" value="0.035"/>   <!-- 70 mm diameter -->
+  <xacro:property name="laser_height" value="0.040"/>   <!-- 40 mm tall     -->
   <!-- ============================================================
        LIDAR JOINT & LINK
@@ -27,5 +28,6 @@
     <parent link="base_link"/>
     <child  link="laser_frame"/>
-    <origin xyz="${laser_x} ${laser_y} ${laser_z}" rpy="0 0 ${laser_yaw}"/>
+    <origin xyz="${laser_x} ${laser_y} ${laser_z}"
+            rpy="0 0 ${laser_yaw}"/>
   </joint>
   <link name="laser_frame">
@@ -47,9 +49,9 @@
     <inertial>
       <origin xyz="0 0 0" rpy="0 0 0"/>
-      <mass value="0.2"/>
+      <mass value="0.200"/>
       <inertia
         ixx="${(1.0/12.0)*0.2*(3*laser_radius*laser_radius + laser_height*laser_height)}"
         iyy="${(1.0/12.0)*0.2*(3*laser_radius*laser_radius + laser_height*laser_height)}"
-        izz="${(1.0/2.0)*0.2*laser_radius*laser_radius}"
+        izz="${(1.0/2.0 )*0.2*laser_radius*laser_radius}"
         ixy="0" iyz="0" ixz="0"/>
     </inertial>

File: description/robot.urdf.xacro (robot description, xacro)
@@ -1,7 +1,20 @@
 <?xml version="1.0"?>
-<robot xmlns:xacro="http://www.ros.org/wiki/xacro"  name="robot">
+<robot xmlns:xacro="http://www.ros.org/wiki/xacro" name="amr4">
+  <!--
+    AMR4 top-level URDF/xacro
+    Platform  : Jetson Orin Nano
+    OS        : Ubuntu 22.04
+    ROS       : ROS 2 Humble
+    Drive     : 4-wheel mecanum (no caster wheels, no camera)
+    Fill-in checklist (search for TODO_FILL):
+      slam.xacro   — chassis size, wheel geometry, wheel positions
+      imu.xacro    — IMU X/Y/Z position on chassis
+      lidar.xacro  — LiDAR X/Y/Z position, yaw
+  -->
+  <!-- Core chassis + 4 wheels -->
   <xacro:include filename="$(find Ros_lidar_bot)/description/slam.xacro"/>
+  <!-- LiDAR link -->
   <xacro:include filename="$(find Ros_lidar_bot)/description/lidar.xacro"/>
-  <xacro:include filename="$(find Ros_lidar_bot)/description/camera.xacro"/>
+  <!-- IMU link -->
   <xacro:include filename="$(find Ros_lidar_bot)/description/imu.xacro"/>
 </robot>

File: description/slam.xacro (robot description, xacro)
@@ -1,32 +1,61 @@
 <?xml version="1.0" ?>
-<robot name="slam" xmlns:xacro="http://www.ros.org/wiki/xacro">
+<robot name="amr4" xmlns:xacro="http://www.ros.org/wiki/xacro">
   <!-- ============================================================
-       CHASSIS & WHEEL DIMENSIONS — FILL IN YOUR VALUES (metres)
+       AMR4 — 4-WHEEL MECANUM DRIVE  (no caster wheels)
+       Jetson Orin Nano · Ubuntu 22.04 · ROS 2 Humble
+       Coordinate convention  (REP-103 / ROS standard):
+         X = forward,  Y = left,  Z = up
+         base_link = centre of the BOTTOM FACE of the chassis box
+       Frame geometry:
+         ground (z=0)
+             │  ← wheel_radius = 0.05 m
+         base_link  (chassis bottom centre)
+             │  ← chassis_height (upward)
+         chassis top
        ============================================================ -->
-  <!-- Chassis box size -->
-  <xacro:property name="chassis_length"  value="0.45"/>   <!-- front-to-back   -->
-  <xacro:property name="chassis_width"   value="0.25"/>   <!-- left-to-right   -->
-  <xacro:property name="chassis_height"  value="0.20"/>   <!-- bottom-to-top   -->
-  <!-- Drive wheel -->
-  <xacro:property name="wheel_radius"    value="0.05035"/>   <!-- RADIUS = 50.35 mm (from sketch) -->
-  <xacro:property name="wheel_width"     value="0.04"/>       <!-- axial thickness -->
-  <!-- X position of wheel axle from robot centre (0 = at centre) -->
-  <xacro:property name="wheel_x"         value="0.0"/>
-  <!-- Half-separation: each wheel is this far from the centre in Y
-       Text said 33cm → 0.165; sketch front-face shows ~35cm → 0.175
-       CONFIRM and update this value! -->
-  <xacro:property name="wheel_half_sep"  value="0.165"/>
-  <!-- Wheel centre height above chassis bottom (base_link) = 11 mm -->
-  <xacro:property name="wheel_z"         value="0.011"/>
-  <!-- Caster wheels -->
-  <xacro:property name="caster_radius"    value="0.019675"/>  <!-- ball caster radius (diameter = 39.35 mm = 50.35 - 11) -->
-  <xacro:property name="caster_front_x"  value="0.12"/>   <!-- front caster X     -->
-  <xacro:property name="caster_rear_x"   value="-0.12"/>   <!-- rear  caster X     -->
-  <!-- ============================================================
-       DERIVED VALUE
-       base_link sits (wheel_radius - wheel_z) above the ground
-       so base_footprint → base_link offset = wheel_radius - wheel_z
-       ============================================================ -->
-  <xacro:property name="ground_to_base"  value="${wheel_radius - wheel_z}"/>
+  <!-- ── CHASSIS SIZE (FILL IN YOUR MEASURED VALUES) ─────────────
+       Measure the outer body of the bot in metres.
+         chassis_length : front-to-back  (X axis)
+         chassis_width  : left-to-right  (Y axis)
+         chassis_height : bottom-to-top  (Z axis)
+       ──────────────────────────────────────────────────────────── -->
+  <xacro:property name="chassis_length"  value="TODO_FILL"/>   <!-- e.g. 0.55  m -->
+  <xacro:property name="chassis_width"   value="TODO_FILL"/>   <!-- e.g. 0.65  m -->
+  <xacro:property name="chassis_height"  value="TODO_FILL"/>   <!-- e.g. 0.15  m -->
+  <!-- ── MECANUM WHEEL DIMENSIONS ────────────────────────────────
+       Sourced from Config.h  (DriveMaster.ino):
+         WHEEL_RADIUS = 0.05 m
+       wheel_width (axial thickness) is not in Config.h — adjust
+       to match your physical wheel (measure the tread width).
+       ──────────────────────────────────────────────────────────── -->
+  <xacro:property name="wheel_radius"    value="0.05"/>         <!-- from Config.h WHEEL_RADIUS -->
+  <xacro:property name="wheel_width"     value="0.05"/>         <!-- axial thickness — adjust to fit -->
+  <!-- ── WHEEL AXLE POSITIONS ─────────────────────────────────────
+       Wheel centre coordinates relative to base_link (metres):
+         X : ±wheel_half_x  (front positive, rear negative)
+         Y : ±wheel_half_y  (left positive, right negative)
+         Z : 0.0  (wheel axle sits at the same height as base_link
+                   because base_link is already wheel_radius above ground)
+       Given by user / confirmed with Config.h CHASSIS_L = 0.52 m:
+         Front-Left  (FL): ( 0.26,  0.32)
+         Front-Right (FR): ( 0.26, -0.32)
+         Rear-Left   (RL): (-0.26,  0.32)
+         Rear-Right  (RR): (-0.26, -0.32)
+       ──────────────────────────────────────────────────────────── -->
+  <xacro:property name="wheel_half_x"   value="0.26"/>          <!-- half wheelbase (front/rear) -->
+  <xacro:property name="wheel_half_y"   value="0.32"/>          <!-- half track width (left/right) -->
+  <!-- Wheel axle Z above base_link.
+       base_link is wheel_radius above ground, so the axle is flush
+       with the chassis bottom face → z = 0. -->
+  <xacro:property name="wheel_z"        value="0.0"/>
+  <!-- ── DERIVED: how high base_link is above ground ─────────────
+       base_footprint → base_link joint rises by wheel_radius so all
+       4 wheels touch the ground plane (z = 0).
+       ──────────────────────────────────────────────────────────── -->
+  <xacro:property name="ground_to_base" value="${wheel_radius}"/>
+  <!-- Mass values — set to 1.0 (dummy); no collision simulation.
+       Update if you ever need realistic dynamics. -->
+  <xacro:property name="chassis_mass"   value="1.0"/>
+  <xacro:property name="wheel_mass"     value="1.0"/>
   <!-- ============================================================
        MATERIALS
@@ -40,6 +69,5 @@
   <link name="base_footprint"/>
   <!-- base_footprint → base_link
-       base_link is at the centre of the BOTTOM FACE of the chassis box.
-       It sits (wheel_radius - wheel_z) above ground so wheels touch ground. -->
+       Rises by wheel_radius so the 4 wheels sit on the ground. -->
   <joint name="base_footprint_joint" type="fixed">
     <parent link="base_footprint"/>
@@ -48,7 +76,7 @@
   </joint>
   <!-- ============================================================
-       base_link / CHASSIS
-       Visual box offset by chassis_height/2 upward so the box
-       sits entirely above base_link (= chassis bottom face centre).
+       base_link / CHASSIS  (cuboid)
+       The visual box is offset +chassis_height/2 in Z so it sits
+       ABOVE base_link (= chassis bottom centre).
        ============================================================ -->
   <link name="base_link">
@@ -67,148 +95,68 @@
     </collision>
     <inertial>
-      <!-- Centre of mass at geometric centre of box -->
       <origin xyz="0 0 ${chassis_height/2}" rpy="0 0 0"/>
-      <mass value="2.0"/>
+      <mass value="${chassis_mass}"/>
       <inertia
-        ixx="${(1.0/12.0)*2.0*(chassis_width*chassis_width + chassis_height*chassis_height)}"
-        iyy="${(1.0/12.0)*2.0*(chassis_length*chassis_length + chassis_height*chassis_height)}"
-        izz="${(1.0/12.0)*2.0*(chassis_length*chassis_length + chassis_width*chassis_width)}"
+        ixx="${(1.0/12.0)*chassis_mass*(chassis_width*chassis_width   + chassis_height*chassis_height)}"
+        iyy="${(1.0/12.0)*chassis_mass*(chassis_length*chassis_length + chassis_height*chassis_height)}"
+        izz="${(1.0/12.0)*chassis_mass*(chassis_length*chassis_length + chassis_width*chassis_width)}"
         ixy="0" iyz="0" ixz="0"/>
     </inertial>
   </link>
   <!-- ============================================================
-       LEFT WHEEL  (positive Y side)
-       Joint origin = physical centre of wheel relative to base_link.
-       Link visual/collision has ZERO local offset → correct TF.
-       Cylinder lies along Z by default; rotate pi/2 about X to align
-       rotation axis with Y-axis.
+       WHEEL MACRO  (cylinder, continuous joint)
+       Cylinder default axis is Z; rotate π/2 about X so the spin
+       axis aligns with Y (the axle / lateral direction).
+       Args:
+         prefix  : fl | fr | rl | rr
+         x_sign  : +1 (front) | -1 (rear)
+         y_sign  : +1 (left)  | -1 (right)
        ============================================================ -->
-  <joint name="left_wheel_joint" type="continuous">
-    <parent link="base_link"/>
-    <child  link="left_wheel"/>
-    <origin xyz="${wheel_x} ${wheel_half_sep} ${wheel_z}" rpy="0 0 0"/>
-    <axis xyz="0 1 0"/>
-  </joint>
-  <link name="left_wheel">
-    <visual>
-      <origin xyz="0 0 0" rpy="${pi/2} 0 0"/>
-      <geometry>
-        <cylinder radius="${wheel_radius}" length="${wheel_width}"/>
-      </geometry>
-      <material name="black"/>
-    </visual>
-    <collision>
-      <origin xyz="0 0 0" rpy="${pi/2} 0 0"/>
-      <geometry>
-        <cylinder radius="${wheel_radius}" length="${wheel_width}"/>
-      </geometry>
-    </collision>
-    <inertial>
-      <origin xyz="0 0 0" rpy="${pi/2} 0 0"/>
-      <mass value="0.5"/>
-      <inertia
-        ixx="${(1.0/12.0)*0.5*(3*wheel_radius*wheel_radius + wheel_width*wheel_width)}"
-        iyy="${(1.0/2.0)*0.5*wheel_radius*wheel_radius}"
-        izz="${(1.0/12.0)*0.5*(3*wheel_radius*wheel_radius + wheel_width*wheel_width)}"
-        ixy="0" iyz="0" ixz="0"/>
-    </inertial>
-  </link>
-  <!-- ============================================================
-       RIGHT WHEEL  (negative Y side)
-       ============================================================ -->
-  <joint name="right_wheel_joint" type="continuous">
-    <parent link="base_link"/>
-    <child  link="right_wheel"/>
-    <origin xyz="${wheel_x} ${-wheel_half_sep} ${wheel_z}" rpy="0 0 0"/>
-    <axis xyz="0 1 0"/>
-  </joint>
-  <link name="right_wheel">
-    <visual>
-      <origin xyz="0 0 0" rpy="${pi/2} 0 0"/>
-      <geometry>
-        <cylinder radius="${wheel_radius}" length="${wheel_width}"/>
-      </geometry>
-      <material name="black"/>
-    </visual>
-    <collision>
-      <origin xyz="0 0 0" rpy="${pi/2} 0 0"/>
-      <geometry>
-        <cylinder radius="${wheel_radius}" length="${wheel_width}"/>
-      </geometry>
-    </collision>
-    <inertial>
-      <origin xyz="0 0 0" rpy="${pi/2} 0 0"/>
-      <mass value="0.5"/>
-      <inertia
-        ixx="${(1.0/12.0)*0.5*(3*wheel_radius*wheel_radius + wheel_width*wheel_width)}"
-        iyy="${(1.0/2.0)*0.5*wheel_radius*wheel_radius}"
-        izz="${(1.0/12.0)*0.5*(3*wheel_radius*wheel_radius + wheel_width*wheel_width)}"
-        ixy="0" iyz="0" ixz="0"/>
-    </inertial>
-  </link>
-  <!-- ============================================================
-       FRONT CASTER  (passive ball caster — fixed joint)
-       ============================================================ -->
-  <joint name="caster_front_joint" type="fixed">
-    <parent link="base_link"/>
-    <child  link="caster_front_link"/>
-    <!-- caster centre sits at wheel ground level; same Z as drive wheel bottom -->
-    <origin xyz="${caster_front_x} 0 ${-caster_radius}" rpy="0 0 0"/>
-  </joint>
-  <link name="caster_front_link">
-    <visual>
-      <origin xyz="0 0 0" rpy="0 0 0"/>
-      <geometry>
-        <sphere radius="${caster_radius}"/>
-      </geometry>
-      <material name="grey"/>
-    </visual>
-    <collision>
-      <origin xyz="0 0 0" rpy="0 0 0"/>
-      <geometry>
-        <sphere radius="${caster_radius}"/>
-      </geometry>
-    </collision>
-    <inertial>
-      <origin xyz="0 0 0" rpy="0 0 0"/>
-      <mass value="0.05"/>
-      <inertia
-        ixx="${(2.0/5.0)*0.05*caster_radius*caster_radius}"
-        iyy="${(2.0/5.0)*0.05*caster_radius*caster_radius}"
-        izz="${(2.0/5.0)*0.05*caster_radius*caster_radius}"
-        ixy="0" iyz="0" ixz="0"/>
-    </inertial>
-  </link>
-  <!-- ============================================================
-       REAR CASTER  (passive ball caster — fixed joint)
-       ============================================================ -->
-  <joint name="caster_rear_joint" type="fixed">
-    <parent link="base_link"/>
-    <child  link="caster_rear_link"/>
-    <origin xyz="${caster_rear_x} 0 ${-caster_radius}" rpy="0 0 0"/>
-  </joint>
-  <link name="caster_rear_link">
-    <visual>
-      <origin xyz="0 0 0" rpy="0 0 0"/>
-      <geometry>
-        <sphere radius="${caster_radius}"/>
-      </geometry>
-      <material name="grey"/>
-    </visual>
-    <collision>
-      <origin xyz="0 0 0" rpy="0 0 0"/>
-      <geometry>
-        <sphere radius="${caster_radius}"/>
-      </geometry>
-    </collision>
-    <inertial>
-      <origin xyz="0 0 0" rpy="0 0 0"/>
-      <mass value="0.05"/>
-      <inertia
-        ixx="${(2.0/5.0)*0.05*caster_radius*caster_radius}"
-        iyy="${(2.0/5.0)*0.05*caster_radius*caster_radius}"
-        izz="${(2.0/5.0)*0.05*caster_radius*caster_radius}"
-        ixy="0" iyz="0" ixz="0"/>
-    </inertial>
-  </link>
+  <xacro:macro name="mecanum_wheel" params="prefix x_sign y_sign">
+    <joint name="${prefix}_wheel_joint" type="continuous">
+      <parent link="base_link"/>
+      <child  link="${prefix}_wheel_link"/>
+      <!-- Wheel centre sits at ±wheel_half_x, ±wheel_half_y, wheel_z (=0)
+           relative to base_link. -->
+      <origin xyz="${x_sign * wheel_half_x} ${y_sign * wheel_half_y} ${wheel_z}"
+              rpy="0 0 0"/>
+      <axis xyz="0 1 0"/>
+      <dynamics damping="0.01" friction="0.1"/>
+    </joint>
+    <link name="${prefix}_wheel_link">
+      <visual>
+        <!-- Rotate the cylinder so its axis aligns with Y (the roll axis) -->
+        <origin xyz="0 0 0" rpy="${pi/2} 0 0"/>
+        <geometry>
+          <cylinder radius="${wheel_radius}" length="${wheel_width}"/>
+        </geometry>
+        <material name="black"/>
+      </visual>
+      <collision>
+        <origin xyz="0 0 0" rpy="${pi/2} 0 0"/>
+        <geometry>
+          <cylinder radius="${wheel_radius}" length="${wheel_width}"/>
+        </geometry>
+      </collision>
+      <inertial>
+        <origin xyz="0 0 0" rpy="${pi/2} 0 0"/>
+        <mass value="${wheel_mass}"/>
+        <!-- Solid cylinder (dummy mass = 1.0, not used for collision) -->
+        <inertia
+          ixx="${(1.0/12.0)*wheel_mass*(3*wheel_radius*wheel_radius + wheel_width*wheel_width)}"
+          iyy="${(1.0/2.0 )*wheel_mass*wheel_radius*wheel_radius}"
+          izz="${(1.0/12.0)*wheel_mass*(3*wheel_radius*wheel_width  + wheel_width*wheel_width)}"
+          ixy="0" iyz="0" ixz="0"/>
+      </inertial>
+    </link>
+  </xacro:macro>
+  <!-- ── Instantiate all 4 wheels ─────────────────────────────── -->
+  <!-- Front-Left  (FL): x= 0.26  y= 0.32 -->
+  <xacro:mecanum_wheel prefix="fl" x_sign=" 1" y_sign=" 1"/>
+  <!-- Front-Right (FR): x= 0.26  y=-0.32 -->
+  <xacro:mecanum_wheel prefix="fr" x_sign=" 1" y_sign="-1"/>
+  <!-- Rear-Left   (RL): x=-0.26  y= 0.32 -->
+  <xacro:mecanum_wheel prefix="rl" x_sign="-1" y_sign=" 1"/>
+  <!-- Rear-Right  (RR): x=-0.26  y=-0.32 -->
+  <xacro:mecanum_wheel prefix="rr" x_sign="-1" y_sign="-1"/>
 </robot>
