Commit message: updated xacro

File: description/imu.xacro (robot description, xacro)
@@ -14,7 +14,7 @@
        ======================================================================= -->
   <!-- IMU position relative to base_link  (FILL IN) -->
-  <xacro:property name="imu_x"  value="TODO_FILL"/>   <!-- e.g.  0.05  -->
-  <xacro:property name="imu_y"  value="TODO_FILL"/>   <!-- e.g.  0.0   -->
-  <xacro:property name="imu_z"  value="TODO_FILL"/>   <!-- e.g.  0.12  -->
+  <xacro:property name="imu_x"  value="0.01"/>   <!-- e.g.  0.05  -->
+  <xacro:property name="imu_y"  value="-0.01"/>   <!-- e.g.  0.0   -->
+  <xacro:property name="imu_z"  value="0.0"/>   <!-- e.g.  0.12  -->
   <!-- IMU orientation offset (FILL IN if the IMU is not mounted flat)
        Leave all zeros if the IMU X axis points robot-forward and Z is up. -->

File: description/lidar.xacro (robot description, xacro)
@@ -14,9 +14,9 @@
        ======================================================================= -->
   <!-- LiDAR position relative to base_link  (FILL IN) -->
-  <xacro:property name="laser_x"      value="TODO_FILL"/>   <!-- e.g.  0.0   -->
-  <xacro:property name="laser_y"      value="TODO_FILL"/>   <!-- e.g.  0.0   -->
-  <xacro:property name="laser_z"      value="TODO_FILL"/>   <!-- e.g.  0.18  (height of LiDAR above chassis bottom) -->
+  <xacro:property name="laser_x"      value="0.0"/>          <!-- chassis centre — adjust to physical mount X -->
+  <xacro:property name="laser_y"      value="0.0"/>          <!-- chassis centre — adjust to physical mount Y -->
+  <xacro:property name="laser_z"      value="0.10"/>         <!-- = chassis_height: LiDAR sits on top of the chassis box -->
   <!-- LiDAR yaw rotation  (FILL IN — see note above) -->
-  <xacro:property name="laser_yaw"    value="TODO_FILL"/>   <!-- 0.0 or ${pi} -->
+  <xacro:property name="laser_yaw"    value="0.0"/>          <!-- 0.0 = LiDAR 0° mark faces robot front (most common) -->
   <!-- LiDAR cylinder visual dimensions  (FILL IN or leave defaults) -->
   <xacro:property name="laser_radius" value="0.035"/>   <!-- 70 mm diameter -->

File: description/slam.xacro (robot description, xacro)
@@ -20,7 +20,7 @@
          chassis_height : bottom-to-top  (Z axis)
        ──────────────────────────────────────────────────────────── -->
-  <xacro:property name="chassis_length"  value="TODO_FILL"/>   <!-- e.g. 0.55  m -->
-  <xacro:property name="chassis_width"   value="TODO_FILL"/>   <!-- e.g. 0.65  m -->
-  <xacro:property name="chassis_height"  value="TODO_FILL"/>   <!-- e.g. 0.15  m -->
+  <xacro:property name="chassis_length"  value="0.85"/>   <!-- e.g. 0.55  m -->
+  <xacro:property name="chassis_width"   value="0.75"/>   <!-- e.g. 0.65  m -->
+  <xacro:property name="chassis_height"  value="0.10"/>   <!-- e.g. 0.15  m -->
   <!-- ── MECANUM WHEEL DIMENSIONS ────────────────────────────────
        Sourced from Config.h  (DriveMaster.ino):
